File: big_muff_r3a/bass/big_muff_r3a_bass.kicad_pcb (KiCad board)
At the start: 2 copper layers, 58.4 x 85.1 mm, 64 parts, among them X1 +, X2 -, X3 COM

Commit message: Big Muff [REV3A]: minor changes
Parts:
- GB1: footprint KCL:B-PP3-HV -> KCL-VIRTUAL:B-PP3-HV
- RP1, RP2, RP3: footprint SBKCL-TH-SL:RPB-20-1x17-1.6-PNL-7.4-2.8 -> SBKCL-TH-SL:RPB-18-1x17-1.6-PNL-7.4-2.8

Commit message: Big Muff [REV3A]: VE1 changed from B013_D1 to B013_E1
Parts:
- VE1: footprint SBEL:B013_D1 -> SBEL:B013_E1
