File: little_angel_chorus_r1a/little_angel_chorus_r1a.kicad_pcb (KiCad board)
At the start: 2 copper layers, 83.8 x 92.7 mm, 70 parts, among them X1 +, X2 -, X3 COM

Commit message: Little Angel Chorus [REV1]: files renamed, gerber added, minor changes
Parts:
- VE1: footprint SBKCL:G0473_little_angel_chorus_r1a -> SBEL:G0473_A1

Commit message: Little Angel Chorus [REV1A]: minor changes
Other:
- board text added: "1. Просверлить в плате 10 отверстий ø1.5 мм под"
- board text removed: "1. Просверлить в плате 12 отверстий ø1.5 мм под"
