File: копка_земли_r1a/standard-tuned/копка_земли_r1a_standard-tuned.kicad_pcb (KiCad board)
At the start: 2 copper layers, 86.4 x 95.3 mm, 63 parts, among them X1 +, X2 -, X3 COM

Commit message: Копка Земли [REV1]: minor changes
Parts:
- R2: value 105 -> X
Other:
- board text added: "1. R2 не устанавливать."

Commit message: Копка Земли [REV1]: minor changes
Parts:
- GB1: footprint KCL:B-PP3-HV -> KCL-VIRTUAL:B-PP3-HV
- VLS1: footprint KCL:VLS-BR -> KCL-VIRTUAL:VLS-BR
- VMH1, VMH2, VMH3, VMH4: footprint KCL:VMH-STA-DA5-PNL-3.0 -> KCL-TH-ML:VMH-STA-DA5-PNL-3.0
