File: тремоло_саши_огородникова_r1b/тремоло_саши_огородникова_r1b.kicad_pcb (KiCad board)
At the start: 2 copper layers, 58.4 x 81.3 mm, 46 parts, among them X1 COM, X2 COM

Commit message: Minor changes
Parts:
- VLS1: footprint KCL:VLS-BR -> KCL-VIRTUAL:VLS-BR
- VMH1, VMH2: footprint KCL:VMH-STA-DA5-PNL-3.0 -> KCL-TH-ML:VMH-STA-DA5-PNL-3.0

Commit message: Minor changes
Parts:
- SA1: footprint KCL-TH-ML:SW-MTS-102-A2-PNL-6.0 -> KCL-TH-ML:SW-MTS-102-A2-3.0-PNL-6.0
