File: crumbwave_multiplexer_r1a/crumbwave_multiplexer_r1a.kicad_pcb (KiCad board)
At the start: 2 copper layers, 86.4 x 78.7 mm, 71 parts, among them X1 COM, X2 COM

Commit message: Latest boards: solder mask clearance, solder mask minimum width, and gerbers modified
Other:
- rule pad_to_mask_clearance: 0.2 -> 0.1
- rule solder_mask_min_width: 0.1 -> 0.2

Commit message: Minor changes
Parts:
- VD1, VD2, VD3: footprint SBKCL-TH-ML:P-SOD-123-OR-DO-35 -> SBKCL-TH-ML:P-SOD-123-OR-DO-35-V1

Commit message: Crumbwave Multiplexer [REV1A]: RPB1.1…RPB1.3 changed
Parts:
- RPB1: value B100K-B100K-B100K -> A100K-B100K-B100K

Commit message: Crumbwave Multiplexer [REV1A]: HL1 changed to FYL-5013URC, IND.R1 value changed to 4.7 kOhm
Parts:
- HL1: value FYL-5013UWC -> FYL-5013URC
- IND.R1: value 103 -> 472
