File: fishtaur_r1a/fishtaur_r1a.kicad_pcb (KiCad board)
At the start: 2 copper layers, 86.4 x 95.3 mm, 81 parts, among them J1 0.6, J2 0.6, J3 0.6, J4 0.6, X1 +, X2 -, X3 COM

Commit message: Fishtaur [REV1]: minor changes
Parts:
- SB1: footprint KCL:SW-PBS-24-302SP-small -> SBKCL:SW-PBS-24-302SP-2.5

Commit message: Fishtaur [REV1]: minor changes
Parts:
- HL1: footprint KCL:LED-ROUND-05.0-UNI-SH-SPACER -> KCL:LED-ROUND-05.0-UNI-SH-SPACER-PNL-5.3

Commit message: Fishtaur [REV1A]: 2.6 mm holes increased to 2.8 mm
Parts:
- RPB1: footprint SBKCL:RPB-18-3x17-DUAL-SINGLE-SINGLE -> SBKCL-TH-SL:RPB-1590BB-18-3x17-DUAL-SINGLE-SINGLE-1.5-PNL-7.4-2.8

Commit message: Fishtaur [REV1A]: R25 and R27 are interchanged on the schematic due to an error on the silkscreen layer
Parts:
- R25: value 472 -> 561
- R27: value 561 -> 472
- moved R25 2.54 mm to (123.2, 138.4), turned to 90 degrees
- moved R27 2.54 mm to (120.7, 138.4), turned to 270 degrees
Connections:
- R25 pad 1: Net-(R25-Pad1) -> Net-(C23-Pad-)
- R25 pad 2: /J1 -> Net-(R25-Pad2)
- R27 pad 1: Net-(C23-Pad-) -> Net-(R27-Pad1)
- R27 pad 2: Net-(R27-Pad2) -> /J1
- RPB1 pad 21: Net-(R25-Pad1) -> Net-(R27-Pad1)
- RPB1 pad 33: Net-(R27-Pad2) -> Net-(R25-Pad2)
Routing:
- net Net-(R27-Pad2): track 5.08 -> 0.00 mm
- net Net-(R27-Pad1): track 0.00 -> 5.08 mm
- net Net-(R25-Pad2): track 0.00 -> 5.08 mm
- net Net-(R25-Pad1): track 5.08 -> 0.00 mm

Commit message: Fishtaur [REV1A]: minor changes
Parts:
- GB1: footprint KCL:B-PP3-HV -> KCL-VIRTUAL:B-PP3-HV
- J1: footprint KCL:J-TH-d0.6-P05.08 -> KCL-TH-SL:J-TH-d0.6-P05.08
- J2, J4: footprint KCL:J-TH-d0.6-P07.62 -> KCL-TH-SL:J-TH-d0.6-P07.62
- J3: footprint KCL:J-TH-d0.6-P06.35 -> KCL-TH-SL:J-TH-d0.6-P06.35
- X1, X2, X3: footprint KCL:CON-PAD-S-1.0-2.0 -> KCL-TH-SL:CON-PAD-S-1.0-2.0
- XS1: footprint KCL:CON-DC-005 -> KCL-TH-SL:CON-DC-005
- XS2, XS3: footprint SBKCL:CON-ST-008X-04-OR-ST-008X-05 -> SBKCL-TH-SL:CON-ST-008X-04-OR-ST-008X-05
Changed lines of the file:
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@@
   (title_block
     (title Fishtaur)
-    (date 2023-04-16)
+    (date 2023-07-15)
     (rev 1A)
     (company "Igor Ivanov")
@@
     (mod_text_size 1 1)
     (mod_text_width 0.15)
-    (pad_size 3 3)
-    (pad_drill 1.5)
+    (pad_size 2 2)
+    (pad_drill 0.7)
     (pad_to_mask_clearance 0.2)
     (solder_mask_min_width 0.1)
@@
     (add_net VREF)
   )
+  (module KCL-VIRTUAL:B-PP3-HV (layer F.Cu)
+    (at 105.41 196.85)
+    (fp_text reference GB1 (at 0 0) (layer F.SilkS) hide
+      (effects (font (size 1 1) (thickness 0.2)))
+    )
+    (fp_text value PP3 (at 0 1.27) (layer F.Fab) hide
+      (effects (font (size 1 1) (thickness 0.2)))
+    )
+    (fp_line (start 24.25 -8.75) (end 24.25 8.75) (layer Dwgs.User) (width 0.2))
+    (fp_line (start -24.25 -8.75) (end -24.25 8.75) (layer Dwgs.User) (width 0.2))
+    (fp_line (start -24.25 8.75) (end 24.25 8.75) (layer Dwgs.User) (width 0.2))
+    (fp_line (start -24.25 -8.75) (end 24.25 -8.75) (layer Dwgs.User) (width 0.2))
+  )
   (module SBKCL-TH-SL:RPB-1590BB-18-3x17-DUAL-SINGLE-SINGLE-1.5-PNL-7.4-2.8 (layer F.Cu)
     (at 105.41 117.04)
@@
       (effects (font (size 1 1) (thickness 0.2)) (justify right))
     )
-    (fp_text user PLS-06 (at -16.51 11.23) (layer F.Fab)
-      (effects (font (size 1 1) (thickness 0.2)))
-    )
-    (fp_text user XP12 (at 8.89 8.69) (layer F.SilkS)
-      (effects (font (size 1 1) (thickness 0.2)) (justify left))
-    )
-    (fp_text user PLS-06 (at 16.51 11.23) (layer F.Fab)
-      (effects (font (size 1 1) (thickness 0.2)))
-    )
-    (fp_text user XP11 (at -8.89 8.69) (layer F.SilkS)
-      (effects (font (size 1 1) (thickness 0.2)) (justify right))
-    )
     (fp_circle (center -7.9 0) (end -6.5 0) (layer Eco1.User) (width 0.4))
     (fp_line (start 24.13 9.96) (end 24.13 12.5) (layer F.CrtYd) (width 0.1))
@@
     (fp_line (start -40.64 12.5) (end -40.64 14) (layer F.CrtYd) (width 0.1))
     (fp_circle (center -40.92 0) (end -39.52 0) (layer Eco1.User) (width 0.4))
+    (fp_text user PLS-06 (at -16.51 11.23) (layer F.Fab)
+      (effects (font (size 1 1) (thickness 0.2)))
+    )
+    (fp_text user XP12 (at 8.89 8.69) (layer F.SilkS)
+      (effects (font (size 1 1) (thickness 0.2)) (justify left))
+    )
+    (fp_text user PLS-06 (at 16.51 11.23) (layer F.Fab)
+      (effects (font (size 1 1) (thickness 0.2)))
+    )
+    (fp_text user XP11 (at -8.89 8.69) (layer F.SilkS)
+      (effects (font (size 1 1) (thickness 0.2)) (justify right))
+    )
     (pad 13 thru_hole rect (at -22.86 11.23) (size 2 2) (drill 1) (layers B.Cu B.Mask)
       (net 21 "Net-(R10-Pad2)"))
@@
     (fp_arc (start 42 54.75) (end 42 51.75) (angle -90) (layer Eco1.User) (width 0.4))
   )
-  (module SBKCL:CON-ST-008X-04-OR-ST-008X-05 (layer F.Cu)
+  (module SBKCL-TH-SL:CON-ST-008X-04-OR-ST-008X-05 (layer F.Cu)
     (at 86.36 100.33 180)
     (fp_text reference XS3 (at 6.35 -13.335 90) (layer F.SilkS)
@@
     (pad "" np_thru_hole circle (at -4.2 -19 180) (size 2.2 2.2) (drill 2.2) (layers *.Cu *.Mask))
   )
-  (module SBKCL:CON-ST-008X-04-OR-ST-008X-05 (layer F.Cu)
+  (module SBKCL-TH-SL:CON-ST-008X-04-OR-ST-008X-05 (layer F.Cu)
     (at 124.46 100.33 180)
     (fp_text reference XS2 (at -6.35 -13.335 90) (layer F.SilkS)
@@
     (pad "" np_thru_hole circle (at -4.2 -19 180) (size 2.2 2.2) (drill 2.2) (layers *.Cu *.Mask))
   )
-  (module KCL:CON-PAD-S-1.0-2.0 (layer F.Cu)
+  (module KCL-TH-SL:CON-PAD-S-1.0-2.0 (layer F.Cu)
     (at 111.76 105.41)
     (fp_text reference X1 (at 0 -1.905) (layer F.SilkS)
@@
     (fp_circle (center 0 0) (end 2.6 0) (layer F.CrtYd) (width 0.1))
   )
-  (module KCL:CON-PAD-S-1.0-2.0 (layer F.Cu)
+  (module KCL-TH-SL:CON-PAD-S-1.0-2.0 (layer F.Cu)
     (at 115.57 105.41)
     (fp_text reference X2 (at 0 -1.905) (layer F.SilkS)
@@
       (net 5 /PP3-NEG))
   )
-  (module KCL:B-PP3-HV (layer F.Cu)
-    (at 105.41 196.85)
-    (fp_text reference GB1 (at 0 0) (layer F.SilkS) hide
-      (effects (font (size 1 1) (thickness 0.2)))
-    )
-    (fp_text value PP3 (at 0 1.27) (layer F.Fab) hide
-      (effects (font (size 1 1) (thickness 0.2)))
-    )
-    (fp_line (start -24.25 -8.75) (end 24.25 -8.75) (layer Dwgs.User) (width 0.2))
-    (fp_line (start -24.25 8.75) (end 24.25 8.75) (layer Dwgs.User) (width 0.2))
-    (fp_line (start -24.25 -8.75) (end -24.25 8.75) (layer Dwgs.User) (width 0.2))
-    (fp_line (start 24.25 -8.75) (end 24.25 8.75) (layer Dwgs.User) (width 0.2))
-  )
   (module KCL:C-DISK-D04.2-T03.0-P05.08-d0.5 (layer F.Cu)
     (at 135.89 107.95)
@@
       (net 1 COM))
   )
-  (module KCL:CON-PAD-S-1.0-2.0 (layer F.Cu)
+  (module KCL-TH-SL:CON-PAD-S-1.0-2.0 (layer F.Cu)
     (at 105.41 186.055)
     (fp_text reference X3 (at 1.27 0) (layer F.SilkS)
@@
       (net 1 COM))
   )
-  (module KCL:CON-DC-005 (layer F.Cu)
+  (module KCL-TH-SL:CON-DC-005 (layer F.Cu)
     (at 105.41 92.71 180)
     (fp_text reference XS1 (at 0 -15.24) (layer F.SilkS)
@@
       (net 10 /J2))
   )
-  (module KCL:J-TH-d0.6-P06.35 (layer F.Cu)
+  (module KCL-TH-SL:J-TH-d0.6-P06.35 (layer F.Cu)
     (at 104.775 133.35)
     (fp_text reference J3 (at 4.445 0) (layer F.SilkS)
@@
     (fp_line (start -4.445 1.27) (end 4.445 1.27) (layer F.SilkS) (width 0.2))
     (fp_line (start -4.445 -1.27) (end 4.445 -1.27) (layer F.SilkS) (width 0.2))
-    (pad J thru_hole rect (at -3.175 0) (size 2 2) (drill 0.7) (layers *.Cu *.Mask)
+    (pad J thru_hole rect (at -3.175 0) (size 2 2) (drill 0.7) (layers B.Cu B.Mask)
       (net 10 /J2))
-    (pad J thru_hole rect (at 3.175 0) (size 2 2) (drill 0.7) (layers *.Cu *.Mask)
+    (pad J thru_hole rect (at 3.175 0) (size 2 2) (drill 0.7) (layers B.Cu B.Mask)
       (net 10 /J2))
   )
@@
       (net 11 /J1))
   )
-  (module KCL:J-TH-d0.6-P05.08 (layer F.Cu)
+  (module KCL-TH-SL:J-TH-d0.6-P05.08 (layer F.Cu)
     (at 84.455 146.05)
     (fp_text reference J1 (at 0 -2.54) (layer F.SilkS)
@@
     (fp_line (start -3.81 1.27) (end 3.81 1.27) (layer F.SilkS) (width 0.2))
     (fp_line (start -3.81 -1.27) (end 3.81 -1.27) (layer F.SilkS) (width 0.2))
-    (pad J thru_hole rect (at -2.54 0) (size 2 2) (drill 0.7) (layers *.Cu *.Mask)
+    (pad J thru_hole rect (at -2.54 0) (size 2 2) (drill 0.7) (layers B.Cu B.Mask)
       (net 11 /J1))
-    (pad J thru_hole rect (at 2.54 0) (size 2 2) (drill 0.7) (layers *.Cu *.Mask)
+    (pad J thru_hole rect (at 2.54 0) (size 2 2) (drill 0.7) (layers B.Cu B.Mask)
       (net 11 /J1))
   )
-  (module KCL:J-TH-d0.6-P07.62 (layer F.Cu)
+  (module KCL-TH-SL:J-TH-d0.6-P07.62 (layer F.Cu)
     (at 93.98 160.02 90)
     (fp_text reference J2 (at -5.08 0 270) (layer F.SilkS)
@@
     (fp_line (start -5.08 1.27) (end 5.08 1.27) (layer F.SilkS) (width 0.2))
     (fp_line (start -5.08 -1.27) (end 5.08 -1.27) (layer F.SilkS) (width 0.2))
-    (pad J thru_hole rect (at -3.81 0 90) (size 2 2) (drill 0.7) (layers *.Cu *.Mask)
+    (pad J thru_hole rect (at -3.81 0 90) (size 2 2) (drill 0.7) (layers B.Cu B.Mask)
       (net 10 /J2))
-    (pad J thru_hole rect (at 3.81 0 90) (size 2 2) (drill 0.7) (layers *.Cu *.Mask)
+    (pad J thru_hole rect (at 3.81 0 90) (size 2 2) (drill 0.7) (layers B.Cu B.Mask)
       (net 10 /J2))
   )
-  (module KCL:J-TH-d0.6-P07.62 (layer F.Cu)
+  (module KCL-TH-SL:J-TH-d0.6-P07.62 (layer F.Cu)
     (at 119.38 151.13)
     (fp_text reference J4 (at 0 2.54) (layer F.SilkS)
@@
     (fp_line (start -5.08 1.27) (end 5.08 1.27) (layer F.SilkS) (width 0.2))
     (fp_line (start -5.08 -1.27) (end 5.08 -1.27) (layer F.SilkS) (width 0.2))
-    (pad J thru_hole rect (at -3.81 0) (size 2 2) (drill 0.7) (layers *.Cu *.Mask)
+    (pad J thru_hole rect (at -3.81 0) (size 2 2) (drill 0.7) (layers B.Cu B.Mask)
       (net 10 /J2))
-    (pad J thru_hole rect (at 3.81 0) (size 2 2) (drill 0.7) (layers *.Cu *.Mask)
+    (pad J thru_hole rect (at 3.81 0) (size 2 2) (drill 0.7) (layers B.Cu B.Mask)
       (net 10 /J2))
   )
@@
   (segment (start 99.06 143.51) (end 102.87 143.51) (width 0.6) (layer B.Cu) (net 22))
   (segment (start 115.57 128.27) (end 115.57 133.35) (width 0.6) (layer B.Cu) (net 23))
-  (segment (start 120.65 128.27) (end 120.65 133.35) (width 0.6) (layer B.Cu) (net 48))
-  (segment (start 123.19 128.27) (end 123.19 133.35) (width 1) (layer B.Cu) (net 47))
   (segment (start 100.33 120.65) (end 100.33 118.11) (width 1) (layer B.Cu) (net 24))
   (segment (start 103.505 130.175) (end 102.87 129.54) (width 1) (layer B.Cu) (net 24))
@@
   (segment (start 92.71 144.145) (end 95.885 144.145) (width 0.6) (layer B.Cu) (net 45))
   (segment (start 123.19 143.51) (end 123.19 147.32) (width 1) (layer B.Cu) (net 46))
+  (segment (start 123.19 128.27) (end 123.19 133.35) (width 1) (layer B.Cu) (net 47))
+  (segment (start 120.65 128.27) (end 120.65 133.35) (width 0.6) (layer B.Cu) (net 48))
   (zone (net 1) (net_name COM) (layer B.Cu) (hatch edge 0.508)
     (connect_pads (clearance 0.6))

Commit message: Fishtaur [REV1A]: minor changes
Parts:
- D1, D2, D3: footprint KCL:P-DIP-08 -> KCL-TH-SL:P-DIP-08
- HL1: footprint KCL:LED-ROUND-05.0-UNI-SH-SPACER-PNL-5.3 -> KCL-TH-SL:LED-ROUND-05.0-UNI-SH-SPACER-PNL-5.3
- VD1, VD2, VD3: footprint KCL:P-DO-41 -> KCL-TH-SL:P-DO-41
- VD4, VD5: footprint KCL:P-DO-7 -> KCL-TH-SL:P-DO-7
- VLS1: footprint KCL:VLS-BR -> KCL-VIRTUAL:VLS-BR

Commit message: Fishtaur [REV1A]: minor changes
Parts:
- SB1: footprint SBKCL:SW-PBS-24-302SP-2.5 -> KCL-TH-SL:SW-PBS-24-302SP-2.5-PNL-13.0
- VMH1, VMH2, VMH3, VMH4: footprint KCL:VMH-STA-DA5 -> KCL-TH-SL:VMH-STA-DA5-PNL-3.0
