File: PCBS-PCAS/ТКП-3.20.A/ТКП-1.20.A-3/ТКП-1.20.A-3.kicad_pcb (KiCad board)
At the start: 2 copper layers, 81.3 x 17.1 mm, 5 parts

Commit message: ТКП-1.20.A 1590BB Potentiometer Board 18 3x17 [REV1A]: project files are moved to cipher-based storage directory
Parts:
- RP1: value RP1: 16/17 -> RP1: B500K
- RP2: value RP2: 16/17 -> RP2: A1K
- RP3: value RP3: 16/17 -> RP3: B100K
