File: PCBS-PCAS/ТКП-3.29.A/ТКП-1.29.A-1/ТКП-1.29.A-1.kicad_pcb (KiCad board)
At the start: 2 copper layers, 55.9 x 17.1 mm, 6 parts

Commit message: ТКП-1.29.A-1 Edamamer Potentiometer Board [REV1A]: some changes
Parts:
- RP1: value RP1: 16/17 -> RP1: A100K
- RP2: value RP2: 16/17 -> RP2: A500K
- RP3: value RP3: 16/17 -> RP3: A500K
