File: PCBS-PCAS/ТКП-3.30.A/ТКП-1.30.A-2/ТКП-1.30.A-2.kicad_pcb (KiCad board)
At the start: 2 copper layers, 58.4 x 85.1 mm, 64 parts, among them X1 +, X2 -, X3 COM

Commit message: ТКП-1.30.A Big Muff [REV3A]: minor changes
Other:
- board text added: "1. VT1...4 установить противоположно шелкографии."
- board text removed: "1. VT1...4 устанавливать противоположно"
- board text removed: "шелкографии."
Changed lines of the file:
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@@
-(kicad_pcb (version 20171130) (host pcbnew 5.1.6-c6e7f7d~87~ubuntu19.10.1)
+(kicad_pcb (version 20171130) (host pcbnew 5.1.12-84ad8e8a86~92~ubuntu20.04.1)
   (general
     (thickness 1.6)
-    (drawings 13)
+    (drawings 12)
     (tracks 224)
     (zones 0)
@@
   (page A4 portrait)
   (title_block
-    (title "Big Muff (Bass)")
-    (date 2023-02-10)
+    (title ТКП-1.30.A-2)
+    (date 2024-01-21)
     (rev 3A)
-    (company "Igor Ivanov")
-    (comment 1 https://github.com/Adept666)
-    (comment 2 "This project is licensed under GNU General Public License v3.0 or later")
+    (company "Big Muff [REV3A] Bass")
+    (comment 1 http://github.com/Adept666)
+    (comment 2 "Igor Ivanov (Игорь Иванов)")
+    (comment 3 -ТТКРЧПДЛ-)
+    (comment 4 "This project is licensed under GNU General Public License v3.0 or later")
   )
   (layers
@@
     (add_net V)
   )
+  (module KCL-TH-SL:CON-PAD-S-1.0-1.9 (layer F.Cu)
+    (at 96.52 104.14)
+    (fp_text reference X1 (at 0 4.445) (layer F.SilkS)
+      (effects (font (size 1 1) (thickness 0.2)))
+    )
+    (fp_text value + (at 0 2.54) (layer F.Fab)
+      (effects (font (size 1 1) (thickness 0.2)))
+    )
+    (fp_circle (center 0 0) (end 0.762 0) (layer F.CrtYd) (width 0.1))
+    (fp_circle (center 0 0) (end 0.762 0) (layer F.SilkS) (width 0.2))
+    (fp_circle (center 0 0) (end 0.5 0) (layer F.Fab) (width 0.2))
+    (pad 1 thru_hole rect (at 0 0) (size 1.9 1.9) (drill 1) (layers B.Cu B.Mask)
+      (net 7 /PP3-POS))
+  )
+  (module KCL-TH-SL:CON-PAD-S-1.0-1.9 (layer F.Cu)
+    (at 124.46 162.56)
+    (fp_text reference X2 (at 0 4.445) (layer F.SilkS)
+      (effects (font (size 1 1) (thickness 0.2)))
+    )
+    (fp_text value - (at 0 2.54) (layer F.Fab)
+      (effects (font (size 1 1) (thickness 0.2)))
+    )
+    (fp_circle (center 0 0) (end 0.762 0) (layer F.CrtYd) (width 0.1))
+    (fp_circle (center 0 0) (end 0.762 0) (layer F.SilkS) (width 0.2))
+    (fp_circle (center 0 0) (end 0.5 0) (layer F.Fab) (width 0.2))
+    (pad 1 thru_hole rect (at 0 0) (size 1.9 1.9) (drill 1) (layers B.Cu B.Mask)
+      (net 8 /PP3-NEG))
+  )
+  (module KCL-TH-SL:CON-PAD-S-1.0-1.9 (layer F.Cu)
+    (at 105.41 176.53)
+    (fp_text reference X3 (at 1.0795 0) (layer F.SilkS)
+      (effects (font (size 1 1) (thickness 0.2)) (justify left))
+    )
+    (fp_text value COM (at 0.635 0) (layer F.Fab)
+      (effects (font (size 1 1) (thickness 0.2)) (justify left))
+    )
+    (fp_circle (center 0 0) (end 0.762 0) (layer F.CrtYd) (width 0.1))
+    (fp_circle (center 0 0) (end 0.762 0) (layer F.SilkS) (width 0.2))
+    (fp_circle (center 0 0) (end 0.5 0) (layer F.Fab) (width 0.2))
+    (pad 1 thru_hole rect (at 0 0) (size 1.9 1.9) (drill 1) (layers B.Cu B.Mask)
+      (net 1 COM))
+  )
   (module SBEL:B013_E1 locked (layer F.Cu)
     (at 105.41 148.59)
@@
       (effects (font (size 1 1) (thickness 0.2)))
     )
-    (fp_arc (start 27.1 52.25) (end 27.1 49) (angle -90) (layer Eco1.User) (width 0.4))
-    (fp_arc (start -27.1 52.25) (end -23.85 52.25) (angle -90) (layer Eco1.User) (width 0.4))
-    (fp_arc (start 27.1 -52.25) (end 23.85 -52.25) (angle -90) (layer Eco1.User) (width 0.4))
-    (fp_arc (start -27.1 -52.25) (end -27.1 -49) (angle -90) (layer Eco1.User) (width 0.4))
     (fp_line (start 23.85 52.25) (end 23.85 55.75) (layer Eco1.User) (width 0.4))
     (fp_line (start -23.85 52.25) (end -23.85 55.75) (layer Eco1.User) (width 0.4))
@@
     (fp_circle (center -43.15 1.27) (end -37.15 1.27) (layer Eco1.User) (width 0.4))
     (fp_circle (center 43.15 1.27) (end 49.15 1.27) (layer Eco1.User) (width 0.4))
+    (fp_arc (start 27.1 52.25) (end 27.1 49) (angle -90) (layer Eco1.User) (width 0.4))
+    (fp_arc (start -27.1 52.25) (end -23.85 52.25) (angle -90) (layer Eco1.User) (width 0.4))
+    (fp_arc (start 27.1 -52.25) (end 23.85 -52.25) (angle -90) (layer Eco1.User) (width 0.4))
+    (fp_arc (start -27.1 -52.25) (end -27.1 -49) (angle -90) (layer Eco1.User) (width 0.4))
   )
   (module KCL-VIRTUAL:B-PP3-HV (layer F.Cu)
@@
       (net 23 "Net-(C13-Pad1)"))
   )
-  (module KCL-TH-SL:CON-PAD-S-1.0-1.9 (layer F.Cu)
-    (at 96.52 104.14)
-    (fp_text reference X1 (at 0 4.445) (layer F.SilkS)
-      (effects (font (size 1 1) (thickness 0.2)))
-    )
-    (fp_text value + (at 0 2.54) (layer F.Fab)
-      (effects (font (size 1 1) (thickness 0.2)))
-    )
-    (fp_circle (center 0 0) (end 0.5 0) (layer F.Fab) (width 0.2))
-    (fp_circle (center 0 0) (end 0.762 0) (layer F.SilkS) (width 0.2))
-    (fp_circle (center 0 0) (end 0.5 0) (layer F.CrtYd) (width 0.1))
-    (pad 1 thru_hole rect (at 0 0) (size 1.9 1.9) (drill 1) (layers B.Cu B.Mask)
-      (net 7 /PP3-POS))
-  )
-  (module KCL-TH-SL:CON-PAD-S-1.0-1.9 (layer F.Cu)
-    (at 124.46 162.56)
-    (fp_text reference X2 (at 0 4.445) (layer F.SilkS)
-      (effects (font (size 1 1) (thickness 0.2)))
-    )
-    (fp_text value - (at 0 2.54) (layer F.Fab)
-      (effects (font (size 1 1) (thickness 0.2)))
-    )
-    (fp_circle (center 0 0) (end 0.5 0) (layer F.CrtYd) (width 0.1))
-    (fp_circle (center 0 0) (end 0.762 0) (layer F.SilkS) (width 0.2))
-    (fp_circle (center 0 0) (end 0.5 0) (layer F.Fab) (width 0.2))
-    (pad 1 thru_hole rect (at 0 0) (size 1.9 1.9) (drill 1) (layers B.Cu B.Mask)
-      (net 8 /PP3-NEG))
-  )
-  (module KCL-TH-SL:CON-PAD-S-1.0-1.9 (layer F.Cu)
-    (at 105.41 176.53)
-    (fp_text reference X3 (at 1.0795 0) (layer F.SilkS)
-      (effects (font (size 1 1) (thickness 0.2)) (justify left))
-    )
-    (fp_text value COM (at 0.635 0) (layer F.Fab)
-      (effects (font (size 1 1) (thickness 0.2)) (justify left))
-    )
-    (fp_circle (center 0 0) (end 0.5 0) (layer F.CrtYd) (width 0.1))
-    (fp_circle (center 0 0) (end 0.762 0) (layer F.SilkS) (width 0.2))
-    (fp_circle (center 0 0) (end 0.5 0) (layer F.Fab) (width 0.2))
-    (pad 1 thru_hole rect (at 0 0) (size 1.9 1.9) (drill 1) (layers B.Cu B.Mask)
-      (net 1 COM))
-  )
   (module KCL-TH-SL:P-TO-92-E-B-C (layer F.Cu)
     (at 123.19 106.68 180)
@@
       (effects (font (size 1 1) (thickness 0.2)))
     )
-    (fp_text value PBS-24-302SP (at 0 7.62) (layer F.Fab)
+    (fp_text value PBS-24-302SP (at 0 0) (layer F.Fab)
       (effects (font (size 1 1) (thickness 0.2)))
     )
@@
       (effects (font (size 1 1) (thickness 0.2)))
     )
-    (fp_text value DC-005 (at 0 -10.795) (layer F.Fab)
+    (fp_text value DC-005 (at 0 -6.985) (layer F.Fab)
       (effects (font (size 1 1) (thickness 0.2)))
     )
@@
       (net 1 COM))
   )
-  (gr_text шелкографии. (at 90.17 250.19) (layer F.Fab)
+  (gr_text "1. VT1...4 установить противоположно шелкографии." (at 90.17 250.19) (layer F.Fab)
     (effects (font (size 2.54 2.54) (thickness 0.2)) (justify left))
   )
-  (gr_text "1. VT1...4 устанавливать противоположно" (at 90.17 246.38) (layer F.Fab)
-    (effects (font (size 2.54 2.54) (thickness 0.2)) (justify left))
-  )
