File: PCBS-PCAS/ТКП-3.13.A/ТКП-1.13.A-2/ТКП-1.13.A-2.kicad_pcb (KiCad board)
At the start: 2 copper layers, 58.4 x 85.1 mm, 63 parts, among them X1 +, X2 -, X3 COM

Commit message: ТКП-1.13.A Big Muff [REV2A]: project files are moved to cipher-based storage directory
Parts:
- C10, C7: value 105 -> 683
- C12: value 392 -> 332
- C15, C5, C6, C9: value 105 -> 104
- R13, R18, R7: value 103 -> 123
- R25: value 202 -> 272
- R6: value 514 -> 474
- R8: value 101 -> 391
- R9: value 182 -> 102
- VD2, VD3, VD4, VD5: value 6263 -> 4148
- VT1, VT2, VT3, VT4: value 5088 -> 547
Other:
- board text added: "2. VT1...4 установить противоположно шелкографии."

Commit message: ТКП-1.13.A Big Muff [REV2A]: minor changes
Parts:
- C10, C12, C13, C14, C15, C2, C3, C5, C6, C7, C9: footprint KCL:C-DISK-D04.2-T03.0-P05.08-d0.5 -> KCL-TH-SL:C-DISK-D04.2-T03.0-P05.08-d0.5
- GB1: footprint KCL:B-PP3-HV -> KCL-VIRTUAL:B-PP3-HV
- X1, X2, X3: footprint KCL:CON-PAD-S-1.0-2.0 -> KCL-TH-SL:CON-PAD-S-1.0-2.0
- XP1: footprint KCL:CON-DC-005S -> KCL-TH-SL:CON-DC-005S
- XS1, XS2: footprint KCL:CON-PJ-644C -> KCL-TH-SL:CON-PJ-644C

Commit message: ТКП-1.13.A Big Muff [REV2A]: minor changes
Parts:
- C1: footprint KCL:CP-RADIAL-D05.0-P02.0-CLS -> KCL-TH-SL:CP-RADIAL-D05.0-P02.0-CLS
- C11, C4, C8: footprint KCL:C-SM-1206 -> KCL-SM:C-SM-1206
- HL1: footprint KCL:LED-ROUND-05.0-UNI-SH-SPACER-PNL-5.3 -> KCL-TH-SL:LED-ROUND-05.0-UNI-SH-SPACER-PNL-5.3
- R1, R2, R3: footprint KCL:R-MFR-12 -> KCL-TH-SL:R-MFR-12
- VD1: footprint KCL:P-DO-41 -> KCL-TH-SL:P-DO-41
- VD2, VD3, VD4, VD5: footprint KCL:P-DO-35 -> KCL-TH-SL:P-DO-35
- VT1, VT2, VT3, VT4: footprint KCL:P-TO-92-E-B-C -> KCL-TH-SL:P-TO-92-E-B-C

Commit message: ТКП-1.13.A Big Muff [REV2A]: minor changes
Parts:
- R10, R11, R12, R13, R14, R15, R16, R17, R18, R19, R20, R21, R22, R23, R24, R25, R4, R5, R6, R7, R8, R9: footprint KCL:R-SM-1206 -> KCL-SM:R-SM-1206
- SB1: footprint KCL:SW-PBS-24-302SP -> KCL-TH-SL:SW-PBS-24-302SP-3.0-PNL-13.0
- VLS1: footprint KCL:VLS-BR -> KCL-VIRTUAL:VLS-BR
Changed lines of the file:
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@@
       (net 18 "Net-(C3-Pad2)"))
   )
-  (module KCL:R-SM-1206 (layer B.Cu)
+  (module KCL-SM:R-SM-1206 (layer B.Cu)
     (at 82.55 116.84)
     (fp_text reference R25 (at -2.54 0) (layer B.SilkS)
@@
       (net 1 COM))
   )
-  (module KCL:R-SM-1206 (layer B.Cu)
+  (module KCL-SM:R-SM-1206 (layer B.Cu)
     (at 92.71 128.27)
     (fp_text reference R24 (at -2.54 0) (layer B.SilkS)
@@
       (net 34 "Net-(C15-Pad1)"))
   )
-  (module KCL:R-SM-1206 (layer B.Cu)
+  (module KCL-SM:R-SM-1206 (layer B.Cu)
     (at 82.55 114.3)
     (fp_text reference R23 (at -2.54 0) (layer B.SilkS)
@@
       (net 1 COM))
   )
-  (module KCL:R-SM-1206 (layer B.Cu)
+  (module KCL-SM:R-SM-1206 (layer B.Cu)
     (at 92.71 130.81)
     (fp_text reference R22 (at 2.54 0) (layer B.SilkS)
@@
       (net 33 "Net-(C14-Pad2)"))
   )
-  (module KCL:R-SM-1206 (layer B.Cu)
+  (module KCL-SM:R-SM-1206 (layer B.Cu)
     (at 118.11 127 90)
     (fp_text reference R21 (at 0 -1.905 90) (layer B.SilkS)
@@
       (net 30 "Net-(C12-Pad2)"))
   )
-  (module KCL:R-SM-1206 (layer B.Cu)
+  (module KCL-SM:R-SM-1206 (layer B.Cu)
     (at 106.68 124.46 270)
     (fp_text reference R20 (at 0 1.905 270) (layer B.SilkS)
@@
       (net 29 "Net-(C11-Pad2)"))
   )
-  (module KCL:R-SM-1206 (layer B.Cu)
+  (module KCL-SM:R-SM-1206 (layer B.Cu)
     (at 120.65 111.76 180)
     (fp_text reference R19 (at 2.54 0) (layer B.SilkS)
@@
       (net 1 COM))
   )
-  (module KCL:R-SM-1206 (layer B.Cu)
+  (module KCL-SM:R-SM-1206 (layer B.Cu)
     (at 97.79 128.27 180)
     (fp_text reference R18 (at 0 1.905) (layer B.SilkS)
@@
       (net 29 "Net-(C11-Pad2)"))
   )
-  (module KCL:R-SM-1206 (layer B.Cu)
+  (module KCL-SM:R-SM-1206 (layer B.Cu)
     (at 111.76 119.38 270)
     (fp_text reference R17 (at -2.54 0 90) (layer B.SilkS)
@@
       (net 27 "Net-(C10-Pad1)"))
   )
-  (module KCL:R-SM-1206 (layer B.Cu)
+  (module KCL-SM:R-SM-1206 (layer B.Cu)
     (at 120.65 114.3 180)
     (fp_text reference R16 (at 2.54 0) (layer B.SilkS)
@@
       (net 1 COM))
   )
-  (module KCL:R-SM-1206 (layer B.Cu)
+  (module KCL-SM:R-SM-1206 (layer B.Cu)
     (at 90.17 111.76)
     (fp_text reference R15 (at 0 -1.905) (layer B.SilkS)
@@
       (net 26 "Net-(C9-Pad2)"))
   )
-  (module KCL:R-SM-1206 (layer B.Cu)
+  (module KCL-SM:R-SM-1206 (layer B.Cu)
     (at 129.54 106.68 180)
     (fp_text reference R14 (at 0 1.905) (layer B.SilkS)
@@
       (net 1 COM))
   )
-  (module KCL:R-SM-1206 (layer B.Cu)
+  (module KCL-SM:R-SM-1206 (layer B.Cu)
     (at 115.57 104.14 180)
     (fp_text reference R13 (at 0 1.905) (layer B.SilkS)
@@
       (net 25 "Net-(C8-Pad2)"))
   )
-  (module KCL:R-SM-1206 (layer B.Cu)
+  (module KCL-SM:R-SM-1206 (layer B.Cu)
     (at 114.3 107.95 90)
     (fp_text reference R12 (at -2.54 0 90) (layer B.SilkS)
@@
       (net 23 "Net-(C7-Pad1)"))
   )
-  (module KCL:R-SM-1206 (layer B.Cu)
+  (module KCL-SM:R-SM-1206 (layer B.Cu)
     (at 129.54 109.22 180)
     (fp_text reference R11 (at 2.54 0) (layer B.SilkS)
@@
       (net 1 COM))
   )
-  (module KCL:R-SM-1206 (layer B.Cu)
+  (module KCL-SM:R-SM-1206 (layer B.Cu)
     (at 129.54 111.76 180)
     (fp_text reference R10 (at 2.54 0) (layer B.SilkS)
@@
       (net 22 "Net-(C6-Pad2)"))
   )
-  (module KCL:R-SM-1206 (layer B.Cu)
+  (module KCL-SM:R-SM-1206 (layer B.Cu)
     (at 120.65 116.84 180)
     (fp_text reference R9 (at 2.54 0) (layer B.SilkS)
@@
       (net 1 COM))
   )
-  (module KCL:R-SM-1206 (layer B.Cu)
+  (module KCL-SM:R-SM-1206 (layer B.Cu)
     (at 125.73 123.19 180)
     (fp_text reference R8 (at 0 1.905) (layer B.SilkS)
@@
       (net 1 COM))
   )
-  (module KCL:R-SM-1206 (layer B.Cu)
+  (module KCL-SM:R-SM-1206 (layer B.Cu)
     (at 121.92 125.73 180)
     (fp_text reference R7 (at 0 1.905) (layer B.SilkS)
@@
       (net 19 "Net-(C4-Pad2)"))
   )
-  (module KCL:R-SM-1206 (layer B.Cu)
+  (module KCL-SM:R-SM-1206 (layer B.Cu)
     (at 129.54 134.62)
     (fp_text reference R6 (at 0 -1.905) (layer B.SilkS)
@@
       (net 18 "Net-(C3-Pad2)"))
   )
-  (module KCL:R-SM-1206 (layer B.Cu)
+  (module KCL-SM:R-SM-1206 (layer B.Cu)
     (at 129.54 137.16 180)
     (fp_text reference R5 (at 0 -1.905) (layer B.SilkS)
@@
       (net 1 COM))
   )
-  (module KCL:R-SM-1206 (layer B.Cu)
+  (module KCL-SM:R-SM-1206 (layer B.Cu)
     (at 116.84 137.16)
     (fp_text reference R4 (at 0 -1.905) (layer B.SilkS)
@@
       (net 14 /PP3-NEG))
   )
-  (module KCL:VLS-BR (layer F.Cu)
+  (module KCL-VIRTUAL:VLS-BR (layer F.Cu)
     (at 105.41 140.97)
     (fp_text reference VLS1 (at 0 5.08) (layer F.SilkS)
@@
       (net 13 /PP3-POS))
   )
-  (module KCL:SW-PBS-24-302SP (layer F.Cu)
+  (module KCL-TH-SL:SW-PBS-24-302SP-3.0-PNL-13.0 (layer F.Cu)
     (at 105.41 167.64)
     (fp_text reference SB1 (at 0 -7.493) (layer F.SilkS)

Commit message: ТКП-1.13.A Big Muff [REV2A]: minor changes
Parts:
- RP1, RP2, RP3: footprint SBKCL-TH-SL:RPB-20-1x17-1.5-PNL-7.4-2.8 -> SBKCL-TH-SL:RPB-18-1x17-1.5-PNL-7.4-2.8
Changed lines of the file:
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@@
     (add_net V)
   )
-  (module SBKCL-TH-SL:RPB-20-1x17-1.5-PNL-7.4-2.8 (layer F.Cu)
+  (module SBKCL-TH-SL:RPB-18-1x17-1.5-PNL-7.4-2.8 (layer F.Cu)
     (at 124.46 108.15)
     (fp_text reference RP3 (at 0 15.04) (layer F.SilkS)
@@
       (net 38 "Net-(R9-Pad2)"))
   )
-  (module SBKCL-TH-SL:RPB-20-1x17-1.5-PNL-7.4-2.8 (layer F.Cu)
+  (module SBKCL-TH-SL:RPB-18-1x17-1.5-PNL-7.4-2.8 (layer F.Cu)
     (at 105.41 121.92)
     (fp_text reference RP2 (at 0 15.24) (layer F.SilkS)
@@
       (net 31 "Net-(C13-Pad1)"))
   )
-  (module SBKCL-TH-SL:RPB-20-1x17-1.5-PNL-7.4-2.8 (layer F.Cu)
+  (module SBKCL-TH-SL:RPB-18-1x17-1.5-PNL-7.4-2.8 (layer F.Cu)
     (at 86.36 108.15)
     (fp_text reference RP1 (at 0 8.69) (layer F.SilkS)
