File: PCBS-PCAS/ТКП-3.17.B/ТКП-1.17.B-1/ТКП-1.17.B-1.kicad_pcb (KiCad board)
At the start: 2 copper layers, 58.4 x 85.1 mm, 66 parts, among them X1 +, X2 -, X3 COM

Commit message: ТКП-1.17.B-1 Deep Blue Delay [REV3B]: VE1 changed from B013_D1 to B013_E1, VLS1 changed from BR-17.8 to BR-12.7, VMH1 and VMH2 changed from DI5M3x20 to DI5M3x18, screws DIN 965 changed to DIN 7985
Parts:
- RP1, RP2, RP3: footprint SBKCL-TH-SL:RPB-20-1x17-1.5-PNL-7.4-2.8 -> SBKCL-TH-SL:RPB-18-1x17-1.5-PNL-7.4-2.8
- VE1: footprint SBEL:B013_D1 -> SBEL:B013_E1
- VLS1: value BR-17.8 -> BR-12.7
- VMH1, VMH2: value DI5M3x20 -> DI5M3x18
Other:
- board text removed: "1. SB1 установить на проставку ТКП-3.35.A."
