File: PCBS-PCAS/ТКП-3.35.A/ТКП-3.35.A.kicad_pcb (KiCad board)
At the start: 2 copper layers, 17 x 13.5 mm, 0 parts

Commit message: ТКП-3.35.A Spacer PBS-24-302SP [REV1A]: minor changes
Other:
- board text added: "1. Толщина 1.5 мм."
Changed lines of the file:
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@@
 (kicad_pcb (version 20171130) (host pcbnew 5.1.12-84ad8e8a86~92~ubuntu20.04.1)
   (general
-    (thickness 1.6)
-    (drawings 13)
+    (thickness 1.5)
+    (drawings 14)
     (tracks 0)
     (zones 0)
@@
   (title_block
     (title ТКП-3.35.A)
-    (date 2023-12-19)
+    (date 2024-09-14)
     (rev 1A)
     (company "Spacer PBS-24-302SP [REV1A]")
@@
   )
   (layers
-    (0 F.Cu jumper)
+    (0 F.Cu signal)
     (31 B.Cu signal)
+    (41 Cmts.User user)
     (44 Edge.Cuts user)
     (45 Margin user)
@@
     (visible_elements 7FFFFFFF)
     (pcbplotparams
-      (layerselection 0x20000_7ffffffe)
+      (layerselection 0x00200_7ffffffe)
       (usegerberextensions false)
       (usegerberattributes false)
@@
       (psa4output false)
       (plotreference false)
-      (plotvalue true)
+      (plotvalue false)
       (plotinvisibletext false)
       (padsonsilk true)
@@
     (uvia_drill 0.1)
   )
+  (gr_text "1. Толщина 1.5 мм." (at 90.17 250.19) (layer Cmts.User)
+    (effects (font (size 2.54 2.54) (thickness 0.2)) (justify left))
+  )
   (gr_circle (center 110.41 152.59) (end 111.06 152.59) (layer Edge.Cuts) (width 0.4))
