File: PCBS-PCAS/ТКП-3.38.A/ТКП-1.36.A-4/ТКП-1.36.A-4.kicad_pcb (KiCad board)
At the start: 2 copper layers, 58.4 x 109.2 mm, 93 parts, among them J1 X, J2 0, J3 0, J4 0, J5 0, J6 0, J7 0, J8 0, J9 X, X1 COM

Commit message: ТКП-1.36.A-3 and ТКП-1.36.A-4: some changes
Parts:
- VLS1: value BR-12.7 -> BR-17.8
- VMH1, VMH2: value DI5M3x18 -> DI5M3x20
- X1: value COM -> X
Changed lines of the file:
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@@
       (effects (font (size 1 1) (thickness 0.2)) (justify left))
     )
-    (fp_text value COM (at 0.635 0) (layer F.Fab)
+    (fp_text value X (at 0.635 0) (layer F.Fab)
       (effects (font (size 1 1) (thickness 0.2)) (justify left))
     )
@@
       (effects (font (size 1 1) (thickness 0.2)))
     )
-    (fp_text value BR-12.7 (at 0 -3.81) (layer F.Fab)
+    (fp_text value BR-17.8 (at 0 -3.81) (layer F.Fab)
       (effects (font (size 1 1) (thickness 0.2)))
     )
@@
       (effects (font (size 1 1) (thickness 0.2)))
     )
-    (fp_text value DI5M3x18 (at 0 0) (layer F.Fab)
+    (fp_text value DI5M3x20 (at 0 0) (layer F.Fab)
       (effects (font (size 1 1) (thickness 0.2)))
     )
@@
       (effects (font (size 1 1) (thickness 0.2)))
     )
-    (fp_text value DI5M3x18 (at 0 0) (layer F.Fab)
-      (effects (font (size 1 1) (thickness 0.2)))
-    )
+    (fp_text value DI5M3x20 (at 0 0) (layer F.Fab)
+      (effects (font (size 1 1) (thickness 0.2)))
+    )

Commit message: ТКП-1.36.A-3 and ТКП-1.36.A-4: some changes
Parts:
- added VE2: ТКП-6.3.3.A2.B1.3-1.B1.E1, SBEPL:ТКП-6.3.3.A2, F.Cu at (105.4, 148.6)
- VE1: value B013 -> ТКП-6.3.1.B1-1; footprint SBEL:B013_F1 -> SBEL:ТКП-6.3.1.B1

Commit message: ТКП-1.36.A-3 and ТКП-1.36.A-4: some changes
Parts:
- RP1, RP2, RP3, RP4, RP5, RP6: footprint SBKCL-TH-ML:RPB-18-1x17-1.6-PNL-7.4-2.8 -> SBKCL-TH-ML:RPB-18-1x17-1.6-PNL-7.2
- SB1: footprint KCL-TH-ML:SW-PBS-24-302SP-2.5-PNL-13.0 -> KCL-TH-ML:SW-PBS-24-302SP-2.5-PNL-12.0

Commit message: ТКП-1.36.A-3 and ТКП-1.36.A-4: some changes, remaining output files added
Parts:
- VE1: value ТКП-6.3.1.B1-1 -> ТКП-6.3.1.A1.B1.A.1-1; footprint SBEL:ТКП-6.3.1.B1 -> SBEPL:ТКП-6.3.1.A1.B1.A
