File: PCBS-PCAS/ТКП-3.26.A/ТКП-1.26.A-1/ТКП-1.26.A-1.kicad_pcb (KiCad board)
At the start: 2 copper layers, 45.7 x 17.1 mm, 3 parts

Commit message: ТКП-1.26.A-1 Тремоло Саши Огородникова Potentiometer Board [REV1A]: some changes, output files updated
Parts:
- RP1: value RP1: 16/17 -> RP1: A100K
- RP2: value RP2: 16/17 -> RP2: A100K
Changed lines of the file:
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@@
   (module KCL-TH-SL:RP-PDB181-K-20-P (layer F.Cu)
     (at 90.17 142.875 180)
-    (fp_text reference RP2 (at 0 -1.27) (layer F.SilkS)
+    (fp_text reference RP2 (at 0 -1.27 180) (layer F.SilkS)
       (effects (font (size 1 1) (thickness 0.2)))
     )
-    (fp_text value "RP2: 16/17" (at 0 -1.27) (layer F.Fab)
+    (fp_text value "RP2: A100K" (at 0 -1.27 180) (layer F.Fab)
       (effects (font (size 1 1) (thickness 0.2)))
     )
+    (fp_line (start -7.3 3.35) (end -7.3 5.35) (layer F.Fab) (width 0.2))
+    (fp_line (start -8.5 3.35) (end -8.5 5.35) (layer F.Fab) (width 0.2))
+    (fp_line (start -8.5 5.35) (end -7.366 5.35) (layer F.Fab) (width 0.2))
+    (fp_line (start 8.5 -6.15) (end 8.5 23.35) (layer F.CrtYd) (width 0.1))
+    (fp_line (start -8.5 -6.15) (end -8.5 23.35) (layer F.CrtYd) (width 0.1))
+    (fp_line (start -8.5 23.35) (end 8.5 23.35) (layer F.CrtYd) (width 0.1))
+    (fp_line (start -8.5 -6.15) (end 8.5 -6.15) (layer F.CrtYd) (width 0.1))
+    (fp_line (start 8.5 -6.15) (end 8.5 0) (layer F.SilkS) (width 0.2))
+    (fp_line (start -8.5 -6.15) (end -8.5 0) (layer F.SilkS) (width 0.2))
+    (fp_line (start -8.5 -6.15) (end 8.5 -6.15) (layer F.SilkS) (width 0.2))
+    (fp_line (start -3.5 9.85) (end 3.5 9.85) (layer F.Fab) (width 0.2))
+    (fp_line (start 3 9.85) (end 3 23.35) (layer F.Fab) (width 0.2))
+    (fp_line (start -3 9.85) (end -3 23.35) (layer F.Fab) (width 0.2))
+    (fp_line (start 3.5 3.35) (end 3.5 9.85) (layer F.Fab) (width 0.2))
+    (fp_line (start -3.5 3.35) (end -3.5 9.85) (layer F.Fab) (width 0.2))
+    (fp_line (start 8.5 -6.15) (end 8.5 3.35) (layer F.Fab) (width 0.2))
+    (fp_line (start -8.5 -6.15) (end -8.5 3.35) (layer F.Fab) (width 0.2))
+    (fp_line (start -3 23.35) (end 3 23.35) (layer F.Fab) (width 0.2))
+    (fp_line (start -8.5 3.35) (end 8.5 3.35) (layer F.Fab) (width 0.2))
     (fp_line (start -8.5 -6.15) (end 8.5 -6.15) (layer F.Fab) (width 0.2))
-    (fp_line (start -8.5 3.35) (end 8.5 3.35) (layer F.Fab) (width 0.2))
-    (fp_line (start -3 23.35) (end 3 23.35) (layer F.Fab) (width 0.2))
-    (fp_line (start -8.5 -6.15) (end -8.5 3.35) (layer F.Fab) (width 0.2))
-    (fp_line (start 8.5 -6.15) (end 8.5 3.35) (layer F.Fab) (width 0.2))
-    (fp_line (start -3.5 3.35) (end -3.5 9.85) (layer F.Fab) (width 0.2))
-    (fp_line (start 3.5 3.35) (end 3.5 9.85) (layer F.Fab) (width 0.2))
-    (fp_line (start -3 9.85) (end -3 23.35) (layer F.Fab) (width 0.2))
-    (fp_line (start 3 9.85) (end 3 23.35) (layer F.Fab) (width 0.2))
-    (fp_line (start -3.5 9.85) (end 3.5 9.85) (layer F.Fab) (width 0.2))
-    (fp_line (start -8.5 -6.15) (end 8.5 -6.15) (layer F.SilkS) (width 0.2))
-    (fp_line (start -8.5 -6.15) (end -8.5 0) (layer F.SilkS) (width 0.2))
-    (fp_line (start 8.5 -6.15) (end 8.5 0) (layer F.SilkS) (width 0.2))
-    (fp_line (start -8.5 -6.15) (end 8.5 -6.15) (layer F.CrtYd) (width 0.1))
-    (fp_line (start -8.5 23.35) (end 8.5 23.35) (layer F.CrtYd) (width 0.1))
-    (fp_line (start -8.5 -6.15) (end -8.5 23.35) (layer F.CrtYd) (width 0.1))
-    (fp_line (start 8.5 -6.15) (end 8.5 23.35) (layer F.CrtYd) (width 0.1))
-    (fp_line (start -8.5 5.35) (end -7.366 5.35) (layer F.Fab) (width 0.2))
-    (fp_line (start -8.5 3.35) (end -8.5 5.35) (layer F.Fab) (width 0.2))
-    (fp_line (start -7.3 3.35) (end -7.3 5.35) (layer F.Fab) (width 0.2))
     (pad 3 thru_hole rect (at 5 0 180) (size 2.5 2.5) (drill 1.2) (layers B.Cu B.Mask)
       (net 4 "Net-(RP2-Pad3)"))
@@
   (module KCL-TH-SL:RP-PDB181-K-20-P (layer F.Cu)
     (at 120.65 142.875 180)
-    (fp_text reference RP1 (at 0 -1.27) (layer F.SilkS)
+    (fp_text reference RP1 (at 0 -1.27 180) (layer F.SilkS)
       (effects (font (size 1 1) (thickness 0.2)))
     )
-    (fp_text value "RP1: 16/17" (at 0 -1.27) (layer F.Fab)
+    (fp_text value "RP1: A100K" (at 0 -1.27 180) (layer F.Fab)
       (effects (font (size 1 1) (thickness 0.2)))
     )
+    (fp_line (start -7.3 3.35) (end -7.3 5.35) (layer F.Fab) (width 0.2))
+    (fp_line (start -8.5 3.35) (end -8.5 5.35) (layer F.Fab) (width 0.2))
+    (fp_line (start -8.5 5.35) (end -7.366 5.35) (layer F.Fab) (width 0.2))
+    (fp_line (start 8.5 -6.15) (end 8.5 23.35) (layer F.CrtYd) (width 0.1))
+    (fp_line (start -8.5 -6.15) (end -8.5 23.35) (layer F.CrtYd) (width 0.1))
+    (fp_line (start -8.5 23.35) (end 8.5 23.35) (layer F.CrtYd) (width 0.1))
+    (fp_line (start -8.5 -6.15) (end 8.5 -6.15) (layer F.CrtYd) (width 0.1))
+    (fp_line (start 8.5 -6.15) (end 8.5 0) (layer F.SilkS) (width 0.2))
+    (fp_line (start -8.5 -6.15) (end -8.5 0) (layer F.SilkS) (width 0.2))
+    (fp_line (start -8.5 -6.15) (end 8.5 -6.15) (layer F.SilkS) (width 0.2))
+    (fp_line (start -3.5 9.85) (end 3.5 9.85) (layer F.Fab) (width 0.2))
+    (fp_line (start 3 9.85) (end 3 23.35) (layer F.Fab) (width 0.2))
+    (fp_line (start -3 9.85) (end -3 23.35) (layer F.Fab) (width 0.2))
+    (fp_line (start 3.5 3.35) (end 3.5 9.85) (layer F.Fab) (width 0.2))
+    (fp_line (start -3.5 3.35) (end -3.5 9.85) (layer F.Fab) (width 0.2))
+    (fp_line (start 8.5 -6.15) (end 8.5 3.35) (layer F.Fab) (width 0.2))
+    (fp_line (start -8.5 -6.15) (end -8.5 3.35) (layer F.Fab) (width 0.2))
+    (fp_line (start -3 23.35) (end 3 23.35) (layer F.Fab) (width 0.2))
+    (fp_line (start -8.5 3.35) (end 8.5 3.35) (layer F.Fab) (width 0.2))
     (fp_line (start -8.5 -6.15) (end 8.5 -6.15) (layer F.Fab) (width 0.2))
-    (fp_line (start -8.5 3.35) (end 8.5 3.35) (layer F.Fab) (width 0.2))
-    (fp_line (start -3 23.35) (end 3 23.35) (layer F.Fab) (width 0.2))
-    (fp_line (start -8.5 -6.15) (end -8.5 3.35) (layer F.Fab) (width 0.2))
-    (fp_line (start 8.5 -6.15) (end 8.5 3.35) (layer F.Fab) (width 0.2))
-    (fp_line (start -3.5 3.35) (end -3.5 9.85) (layer F.Fab) (width 0.2))
-    (fp_line (start 3.5 3.35) (end 3.5 9.85) (layer F.Fab) (width 0.2))
-    (fp_line (start -3 9.85) (end -3 23.35) (layer F.Fab) (width 0.2))
-    (fp_line (start 3 9.85) (end 3 23.35) (layer F.Fab) (width 0.2))
-    (fp_line (start -3.5 9.85) (end 3.5 9.85) (layer F.Fab) (width 0.2))
-    (fp_line (start -8.5 -6.15) (end 8.5 -6.15) (layer F.SilkS) (width 0.2))
-    (fp_line (start -8.5 -6.15) (end -8.5 0) (layer F.SilkS) (width 0.2))
-    (fp_line (start 8.5 -6.15) (end 8.5 0) (layer F.SilkS) (width 0.2))
-    (fp_line (start -8.5 -6.15) (end 8.5 -6.15) (layer F.CrtYd) (width 0.1))
-    (fp_line (start -8.5 23.35) (end 8.5 23.35) (layer F.CrtYd) (width 0.1))
-    (fp_line (start -8.5 -6.15) (end -8.5 23.35) (layer F.CrtYd) (width 0.1))
-    (fp_line (start 8.5 -6.15) (end 8.5 23.35) (layer F.CrtYd) (width 0.1))
-    (fp_line (start -8.5 5.35) (end -7.366 5.35) (layer F.Fab) (width 0.2))
-    (fp_line (start -8.5 3.35) (end -8.5 5.35) (layer F.Fab) (width 0.2))
-    (fp_line (start -7.3 3.35) (end -7.3 5.35) (layer F.Fab) (width 0.2))
     (pad 3 thru_hole rect (at 5 0 180) (size 2.5 2.5) (drill 1.2) (layers B.Cu B.Mask)
       (net 1 "Net-(RP1-Pad3)"))
@@
       (effects (font (size 1 1) (thickness 0.2)))
     )
+    (fp_line (start 7.62 -0.45) (end 7.62 10.16) (layer F.CrtYd) (width 0.1))
+    (fp_line (start -7.62 -0.45) (end -7.62 10.16) (layer F.CrtYd) (width 0.1))
+    (fp_line (start -7.62 10.16) (end 7.62 10.16) (layer F.CrtYd) (width 0.1))
+    (fp_line (start -7.62 -0.45) (end 7.62 -0.45) (layer F.CrtYd) (width 0.1))
+    (fp_line (start 7.62 1.76) (end 7.62 7.62) (layer F.SilkS) (width 0.2))
+    (fp_line (start -7.62 1.76) (end -7.62 7.62) (layer F.SilkS) (width 0.2))
+    (fp_line (start -7.62 1.76) (end 7.62 1.76) (layer F.SilkS) (width 0.2))
+    (fp_line (start -7.62 1.76) (end 7.62 1.76) (layer F.Fab) (width 0.2))
+    (fp_line (start -7.62 10.16) (end 7.62 10.16) (layer F.Fab) (width 0.2))
+    (fp_line (start -7.62 1.76) (end -7.62 10.16) (layer F.Fab) (width 0.2))
     (fp_line (start 7.62 1.76) (end 7.62 10.16) (layer F.Fab) (width 0.2))
-    (fp_line (start -7.62 1.76) (end -7.62 10.16) (layer F.Fab) (width 0.2))
-    (fp_line (start -7.62 10.16) (end 7.62 10.16) (layer F.Fab) (width 0.2))
-    (fp_line (start -7.62 1.76) (end 7.62 1.76) (layer F.Fab) (width 0.2))
-    (fp_line (start -7.62 1.76) (end 7.62 1.76) (layer F.SilkS) (width 0.2))
-    (fp_line (start -7.62 1.76) (end -7.62 7.62) (layer F.SilkS) (width 0.2))
-    (fp_line (start 7.62 1.76) (end 7.62 7.62) (layer F.SilkS) (width 0.2))
-    (fp_line (start -7.62 -0.45) (end 7.62 -0.45) (layer F.CrtYd) (width 0.1))
-    (fp_line (start -7.62 10.16) (end 7.62 10.16) (layer F.CrtYd) (width 0.1))
-    (fp_line (start -7.62 -0.45) (end -7.62 10.16) (layer F.CrtYd) (width 0.1))
-    (fp_line (start 7.62 -0.45) (end 7.62 10.16) (layer F.CrtYd) (width 0.1))
     (pad 6 thru_hole rect (at 6.35 0) (size 2 2) (drill 0.9) (layers B.Cu B.Mask)
       (net 1 "Net-(RP1-Pad3)"))
