File: PCBS-PCAS/ТКП-3.39.A/ТКП-1.37.A-3/ТКП-1.37.A-3.kicad_pcb (KiCad board)
At the start: 2 copper layers, 58.4 x 81.3 mm, 118 parts, among them J1 X, J10 X, J2 0, J3 X, J4 X, J5 0, J6 0, J7 0, J8 0, J9 0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

Commit message: ТКП-1.37.A Little Angel Chorus [REV2A]: minor changes
Other:
- board text added: "1. DWS.J2, DWS.J3, OC.J1, OC.J3 и OC.J5 оставить"
- board text added: "1. Перечёркнутые элементы не устанавливать."
- board text added: "2. DWS.J1, DWS.J4, OC.J2 и OC.J4 замкнуть."
- board text added: "2. Установить либо PS.C1, либо PS.C2."
- board text added: "3. Установить либо PS.C4, либо PS.C5."
- board text added: "разомкнутыми."
Changed lines of the file:
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@@
   (general
     (thickness 1.6)
-    (drawings 11)
+    (drawings 17)
     (tracks 645)
     (zones 0)
@@
   (title_block
     (title "Little Angel Chorus/Vibrato")
-    (date 2023-04-06)
+    (date 2023-08-26)
     (rev 2A)
     (company "Igor Ivanov")
@@
       (net 4 V))
   )
+  (gr_text "1. DWS.J2, DWS.J3, OC.J1, OC.J3 и OC.J5 оставить" (at 119.83 242.57) (layer B.Fab)
+    (effects (font (size 2.54 2.54) (thickness 0.2)) (justify left mirror))
+  )
+  (gr_text разомкнутыми. (at 119.83 246.38) (layer B.Fab)
+    (effects (font (size 2.54 2.54) (thickness 0.2)) (justify left mirror))
+  )
+  (gr_text "2. DWS.J1, DWS.J4, OC.J2 и OC.J4 замкнуть." (at 119.83 250.19) (layer B.Fab)
+    (effects (font (size 2.54 2.54) (thickness 0.2)) (justify left mirror))
+  )
+  (gr_text "1. Перечёркнутые элементы не устанавливать." (at 90.17 242.57) (layer F.Fab)
+    (effects (font (size 2.54 2.54) (thickness 0.2)) (justify left))
+  )
+  (gr_text "2. Установить либо PS.C1, либо PS.C2." (at 90.17 246.38) (layer F.Fab)
+    (effects (font (size 2.54 2.54) (thickness 0.2)) (justify left))
+  )
+  (gr_text "3. Установить либо PS.C4, либо PS.C5." (at 90.17 250.19) (layer F.Fab)
+    (effects (font (size 2.54 2.54) (thickness 0.2)) (justify left))
+  )
   (gr_text C (at 109.22 173.355) (layer F.SilkS)

Commit message: ТКП-1.37.A Little Angel Chorus [REV2A]: minor changes
Other:
- board text added: "2. Установить либо AL.C1, либо AL.C2."
- board text added: "3. Установить либо PS.C1, либо PS.C2."
- board text added: "4. Установить либо PS.C4, либо PS.C5."
- board text removed: "2. Установить либо PS.C1, либо PS.C2."
- board text removed: "3. Установить либо PS.C4, либо PS.C5."

Commit message: ТКП-1.37.A Little Angel Chorus [REV2A]: DWS.R1 and L.R6 values changed to X
Parts:
- DWS.R1, L.R6: value 0 -> X

Commit message: ТКП-1.37.A-3 Little Angel Chorus/Vibrato [REV2A]: DWS.R1 and L.R6 values changed from X to 0, RPB1.1 and RPB1.2 replaced from R16K1-L15KC B50K to RV16AF-20-15K C50K
Parts:
- DWS.R1, L.R6: value X -> 0
- RPB1: value B50K-B50K -> C50K-C50K
