File: PCBS-PCAS/ТКП-3.39.A/ТКП-1.37.A-1/ТКП-1.37.A-1.kicad_pcb (KiCad board)
At the start: 2 copper layers, 58.4 x 81.3 mm, 118 parts, among them J1 X, J10 X, J2 0, J3 X, J4 X, J5 0, J6 0, J7 0, J8 0, J9 0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

Commit message: ТКП-1.37.A Little Angel Chorus [REV2A]: minor changes
Other:
- board text added: "1. DWS.J1...4, OC.J1, OC.J2, OC.J4 и OC.J5 оставить"
- board text added: "1. Перечёркнутые элементы не устанавливать."
- board text added: "2. OC.J3 замкнуть."
- board text added: "2. Установить либо AL.C1, либо AL.C2."
- board text added: "3. Установить либо PS.C1, либо PS.C2."
- board text added: "4. Установить либо PS.C4, либо PS.C5."
- board text added: "разомкнутыми."

Commit message: ТКП-1.37.A Little Angel Chorus [REV2A]: DWS.R1 and L.R6 values changed to X
Parts:
- DWS.R1, L.R6: value 0 -> X

Commit message: ТКП-1.37.A-1 Little Angel Chorus [REV2A]: DWS.R1 and L.R6 values changed from X to 0, RPB1.1 and RPB1.2 replaced from R16K1-L15KC B50K to RV16AF-20-15K C50K
Parts:
- DWS.R1, L.R6: value X -> 0
- RPB1: value B50K-B50K -> C50K-C50K
