File: PCBS-PCAS/ТКП-3.39.A/ТКП-1.37.A-2/ТКП-1.37.A-2.kicad_pcb (KiCad board)
At the start: 2 copper layers, 58.4 x 81.3 mm, 118 parts, among them J1 X, J10 X, J2 0, J3 X, J4 X, J5 0, J6 0, J7 X, J8 0, J9 0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

Commit message: ТКП-1.37.A Little Angel Chorus [REV2A]: minor changes
Other:
- board text added: "1. DWS.J1...4 и OC.J1...5 оставить разомкнутыми."
- board text added: "1. Перечёркнутые элементы не устанавливать."
- board text added: "2. Установить либо PS.C1, либо PS.C2."
- board text added: "3. Установить либо PS.C4, либо PS.C5."

Commit message: ТКП-1.37.A Little Angel Chorus [REV2A]: minor changes
Other:
- board text added: "2. Установить либо AL.C1, либо AL.C2."
- board text added: "3. Установить либо PS.C1, либо PS.C2."
- board text added: "4. Установить либо PS.C4, либо PS.C5."
- board text removed: "2. Установить либо PS.C1, либо PS.C2."
- board text removed: "3. Установить либо PS.C4, либо PS.C5."
Changed lines of the file:
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@@
   (general
     (thickness 1.6)
-    (drawings 15)
+    (drawings 16)
     (tracks 645)
     (zones 0)
@@
   (title_block
     (title ТКП-1.37.A-2)
-    (date 2023-08-26)
+    (date 2023-08-27)
     (rev 2A)
     (company "Big Devil Vibrato [REV2A]")
@@
       (net 4 V))
   )
+  (gr_text "4. Установить либо PS.C4, либо PS.C5." (at 90.17 250.19) (layer F.Fab)
+    (effects (font (size 2.54 2.54) (thickness 0.2)) (justify left))
+  )
   (gr_text "1. DWS.J1...4 и OC.J1...5 оставить разомкнутыми." (at 119.83 250.19) (layer B.Fab)
     (effects (font (size 2.54 2.54) (thickness 0.2)) (justify left mirror))
   )
-  (gr_text "1. Перечёркнутые элементы не устанавливать." (at 90.17 242.57) (layer F.Fab)
+  (gr_text "1. Перечёркнутые элементы не устанавливать." (at 90.17 238.76) (layer F.Fab)
     (effects (font (size 2.54 2.54) (thickness 0.2)) (justify left))
   )
-  (gr_text "2. Установить либо PS.C1, либо PS.C2." (at 90.17 246.38) (layer F.Fab)
+  (gr_text "2. Установить либо AL.C1, либо AL.C2." (at 90.17 242.57) (layer F.Fab)
     (effects (font (size 2.54 2.54) (thickness 0.2)) (justify left))
   )
-  (gr_text "3. Установить либо PS.C4, либо PS.C5." (at 90.17 250.19) (layer F.Fab)
+  (gr_text "3. Установить либо PS.C1, либо PS.C2." (at 90.17 246.38) (layer F.Fab)
     (effects (font (size 2.54 2.54) (thickness 0.2)) (justify left))
   )

Commit message: ТКП-1.37.A Little Angel Chorus [REV2A]: DWS.R1 and L.R6 values changed to X
Parts:
- DWS.R1, L.R6: value 0 -> X
Changed lines of the file:
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@@
   (title_block
     (title ТКП-1.37.A-2)
-    (date 2023-08-27)
+    (date 2023-11-05)
     (rev 2A)
     (company "Big Devil Vibrato [REV2A]")
@@
       (effects (font (size 0.8 0.8) (thickness 0.2)))
     )
-    (fp_text value 0 (at 0 0 90) (layer F.Fab)
+    (fp_text value X (at 0 0 90) (layer F.Fab)
       (effects (font (size 1 1) (thickness 0.2)))
     )
@@
       (effects (font (size 0.8 0.8) (thickness 0.2)))
     )
-    (fp_text value 0 (at 0 0 90) (layer F.Fab)
-      (effects (font (size 1 1) (thickness 0.2)))
-    )
+    (fp_text value X (at 0 0 90) (layer F.Fab)
+      (effects (font (size 1 1) (thickness 0.2)))
+    )

Commit message: ТКП-1.37.A-2 Big Devil Vibrato [REV2A]: DWS.R1 and L.R6 values changed from X to 0, RPB1.1 and RPB1.2 replaced from R16K1-L15KC B50K to RV16AF-20-15K C50K
Parts:
- DWS.R1, L.R6: value X -> 0
- RPB1: value B50K-B50K -> C50K-C50K
