File: PCBS-PCAS/ТКП-3.17.B/ТКП-1.17.B-2/ТКП-1.17.B-2.kicad_pcb (KiCad board)
At the start: 2 copper layers, 58.4 x 85.1 mm, 67 parts, among them X1 X, X2 X, X3 X

Commit message: ТКП-1.17.B-2 Deep Blue Delay [REV3B] SM: VE1 replaced from ТКП-6.3.1.A1-1 with ТКП-6.3.1.A2.A1.A.1-1, VE2 cipher changed from ТКП-6.3.3.A1-1 to ТКП-6.3.3.A1.A1.2-1.A1.00
Parts:
- VE1: value ТКП-6.3.1.A1-1 -> ТКП-6.3.1.A2.A1.A.1-1; footprint SBEL:ТКП-6.3.1.A1 -> SBEPL:ТКП-6.3.1.A2.A1.A
- VE2: value ТКП-6.3.3.A1-1 -> ТКП-6.3.3.A1.A1.2-1.A1.00; footprint SBEL:ТКП-6.3.3 -> SBEPL:ТКП-6.3.3.A1

Commit message: ТКП-1.17.B-2 Deep Blue Delay [REV3B] SM: RP1…3 replaced from R16K1-L20F with PDB181-K415F, VE2 cipher changed from ТКП-6.3.3.A1.A1.2-1.A1.00 to ТКП-6.3.3.A1.A1.3-1.A1.00
Parts:
- VE2: value ТКП-6.3.3.A1.A1.2-1.A1.00 -> ТКП-6.3.3.A1.A1.3-1.A1.00
