File: PCBS-PCAS/ТКП-3.30.B/ТКП-1.30.B-3/ТКП-1.30.B-3.kicad_pcb (KiCad board)
At the start: 2 copper layers, 58.4 x 85.1 mm, 74 parts, among them X1 X, X2 X, X3 X

Commit message: ТКП-1.30.B-3 and ТКП-1.30.B-4: VE2 cipher changed from ТКП-6.3.3.A1.A1.2-1.A1.00 to ТКП-6.3.3.A1.A1.3-1.A1.00
Parts:
- RP1, RP2, RP3: footprint SBKCL-TH-ML:RPB-18-1x17-1.6-PNL-7.4-2.8 -> SBKCL-TH-ML:RPB-18-1x17-1.6-PNL-7.2
- SB1: footprint KCL-TH-ML:SW-PBS-24-302SP-2.5-PNL-13.0 -> KCL-TH-ML:SW-PBS-24-302SP-2.5-PNL-12.0
- VE2: value ТКП-6.3.3.A1.A1.2-1.A1.00 -> ТКП-6.3.3.A1.A1.3-1.A1.00
