File: PCBS-PCAS/ТКП-3.30.A/ТКП-1.30.A-3/ТКП-1.30.A-3.kicad_pcb (KiCad board)
At the start: 2 copper layers, 58.4 x 85.1 mm, 64 parts, among them X1 X, X2 X, X3 X

Commit message: ТКП-1.30.A-3 and ТКП-1.30.A-4: VE1 changed, VE2 added, washers removed, remaining output files added
Parts:
- added VE2: ТКП-6.3.3.A1-1, SBEL:ТКП-6.3.3, F.Cu at (105.4, 148.6)
- VE1: value B013 -> ТКП-6.3.1.A1-1; footprint SBEL:B013_E1 -> SBEL:ТКП-6.3.1.A1

Commit message: ТКП-1.30.A-3 and ТКП-1.30.A-4: spacer ТКП-3.35.A removed, other minor changes
Parts:
- RP1, RP2, RP3: footprint SBKCL-TH-SL:RPB-18-1x17-1.6-PNL-7.4-2.8 -> SBKCL-TH-SL:RPB-18-1x17-1.6-PNL-7.2
- SB1: footprint KCL-TH-SL:SW-PBS-24-302SP-2.5-PNL-13.0 -> KCL-TH-SL:SW-PBS-24-302SP-2.5-PNL-12.0
Other:
- board text added: "1. X1...3 не устанавливать."
- board text removed: "1. SB1 установить на проставку ТКП-3.35.A."
- board text removed: "2. X1...3 не устанавливать."

Commit message: ТКП-1.30.A-3 Big Muff [REV3A] NYC SM: RP1…3 replaced from R16K1-L20KC with PDB181-K420K, VE1 replaced from ТКП-6.3.1.A1-1 with ТКП-6.3.1.A2.A1.A.1-1, VE2 cipher changed from ТКП-6.3.3.A1-1 to ТКП-6.3.3.A1.A1.2-1.A1.00
Parts:
- VE1: value ТКП-6.3.1.A1-1 -> ТКП-6.3.1.A2.A1.A.1-1; footprint SBEL:ТКП-6.3.1.A1 -> SBEPL:ТКП-6.3.1.A2.A1.A
- VE2: value ТКП-6.3.3.A1-1 -> ТКП-6.3.3.A1.A1.2-1.A1.00; footprint SBEL:ТКП-6.3.3 -> SBEPL:ТКП-6.3.3.A1

Commit message: ТКП-1.30.A-3 and ТКП-1.30.A-4: VE2 cipher changed from ТКП-6.3.3.A1.A1.2-1.A1.00 to ТКП-6.3.3.A1.A1.3-1.A1.00
Parts:
- VE2: value ТКП-6.3.3.A1.A1.2-1.A1.00 -> ТКП-6.3.3.A1.A1.3-1.A1.00
