File: PCBS-PCAS/ТКП-3.21.A/ТКП-1.21.A-2/ТКП-1.21.A-2.kicad_pcb (KiCad board)
At the start: 2 copper layers, 86.4 x 95.3 mm, 81 parts, among them J1 0.6, J2 0.6, J3 0.6, J4 0.6, X1 X, X2 X, X3 COM

Commit message: Minor changes
Parts:
- GB1: value PP3 -> X
Other:
- board text added: "1. SB1 установить на проставку ТКП-3.35.A."
- board text added: "2. X1 и X2 не устанавливать."
Changed lines of the file:
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@@
   (general
     (thickness 1.6)
-    (drawings 9)
+    (drawings 11)
     (tracks 445)
     (zones 0)
@@
   (title_block
     (title ТКП-1.21.A-2)
-    (date 2023-07-15)
+    (date 2023-07-16)
     (rev 1A)
     (company "Fishtaur [REV1A] SM")
@@
       (effects (font (size 1 1) (thickness 0.2)))
     )
-    (fp_text value PP3 (at 0 1.27) (layer F.Fab) hide
+    (fp_text value X (at 0 1.27) (layer F.Fab) hide
       (effects (font (size 1 1) (thickness 0.2)))
     )
@@
       (effects (font (size 1 1) (thickness 0.2)) (justify left))
     )
-    (fp_text value COM (at -1.27 0) (layer F.Fab)
-      (effects (font (size 1 1) (thickness 0.2)) (justify right))
+    (fp_text value COM (at 0.635 0) (layer F.Fab)
+      (effects (font (size 1 1) (thickness 0.2)) (justify left))
     )
     (fp_circle (center 0 0) (end 0.5 0) (layer F.CrtYd) (width 0.1))
@@
       (effects (font (size 1 1) (thickness 0.2)) (justify left))
     )
-    (fp_text value 0.6 (at 0 0) (layer F.Fab)
+    (fp_text value 0.6 (at 0 -0.9525) (layer F.Fab)
       (effects (font (size 1 1) (thickness 0.2)))
     )
@@
       (effects (font (size 1 1) (thickness 0.2)))
     )
-    (fp_text value 0.6 (at 0 0) (layer F.Fab)
+    (fp_text value 0.6 (at 0 -0.9525) (layer F.Fab)
       (effects (font (size 1 1) (thickness 0.2)))
     )
@@
       (effects (font (size 1 1) (thickness 0.2)) (justify right))
     )
-    (fp_text value 0.6 (at 0 0 270) (layer F.Fab)
+    (fp_text value 0.6 (at 0 -0.9525 270) (layer F.Fab)
       (effects (font (size 1 1) (thickness 0.2)))
     )
@@
       (effects (font (size 1 1) (thickness 0.2)))
     )
-    (fp_text value 0.6 (at 0 0) (layer F.Fab)
+    (fp_text value 0.6 (at 0 0.9525) (layer F.Fab)
       (effects (font (size 1 1) (thickness 0.2)))
     )
@@
       (net 16 VB))
   )
+  (gr_text "2. X1 и X2 не устанавливать." (at 90.17 250.19) (layer F.Fab)
+    (effects (font (size 2.54 2.54) (thickness 0.2)) (justify left))
+  )
+  (gr_text "1. SB1 установить на проставку ТКП-3.35.A." (at 90.17 246.38) (layer F.Fab)
+    (effects (font (size 2.54 2.54) (thickness 0.2)) (justify left))
+  )
   (gr_line (start 138.43 92.71) (end 148.59 102.87) (layer Edge.Cuts) (width 0.4))

Commit message: ТКП-1.19.B-2, ТКП-1.21.A-2, ТКП-1.24.B-3, and ТКП-1.24.B-4: 1590BB enclosures changed to custom enclosures
Parts:
- added VE2: ТКП-6.1.3.B1-1, SBEL:ТКП-6.1.3, F.Cu at (105.4, 148.6)
- VE1: value 1590BB -> ТКП-6.1.1.A1-2; footprint SBEL:1590BB_B1 -> SBEL:ТКП-6.1.1.A1

Commit message: ТКП-1.19.B-2, ТКП-1.21.A-2, ТКП-1.24.B-3, and ТКП-1.24.B-4: hole diameters changed
Parts:
- RPB1: footprint SBKCL-TH-SL:RPB-1590BB-18-3x17-DUAL-SINGLE-SINGLE-1.5-PNL-7.4-2.8 -> SBKCL-TH-SL:RPB-1590BB-18-3x17-DUAL-SINGLE-SINGLE-1.5-PNL-7.2
- SB1: footprint KCL-TH-SL:SW-PBS-24-302SP-2.5-PNL-13.0 -> KCL-TH-SL:SW-PBS-24-302SP-2.5-PNL-12.0
Changed lines of the file:
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@@
     (fp_line (start 24.25 -8.75) (end 24.25 8.75) (layer Dwgs.User) (width 0.2))
   )
-  (module SBKCL-TH-SL:RPB-1590BB-18-3x17-DUAL-SINGLE-SINGLE-1.5-PNL-7.4-2.8 (layer F.Cu)
+  (module SBKCL-TH-SL:RPB-1590BB-18-3x17-DUAL-SINGLE-SINGLE-1.5-PNL-7.2 (layer F.Cu)
     (at 105.41 117.04)
     (fp_text reference RPB1 (at 40.64 15.04) (layer F.SilkS)
@@
       (effects (font (size 1 1) (thickness 0.2)) (justify right))
     )
-    (fp_circle (center -40.92 0) (end -39.52 0) (layer Eco1.User) (width 0.4))
     (fp_line (start -40.64 12.5) (end -40.64 14) (layer F.CrtYd) (width 0.1))
     (fp_line (start -40.32 -1.4) (end -40.32 1.4) (layer Dwgs.User) (width 0.2))
@@
     (fp_line (start -40.64 12.5) (end -40.64 14) (layer F.SilkS) (width 0.2))
     (fp_circle (center -33.02 0) (end -29.52 0) (layer Dwgs.User) (width 0.2))
-    (fp_circle (center -33.02 0) (end -29.32 0) (layer Eco1.User) (width 0.4))
+    (fp_circle (center -33.02 0) (end -29.42 0) (layer Eco1.User) (width 0.4))
     (fp_circle (center -33.02 0) (end -30.02 0) (layer Dwgs.User) (width 0.2))
     (fp_line (start -25.52 4) (end -25.52 12.5) (layer Dwgs.User) (width 0.2))
-    (fp_circle (center 25.12 0) (end 26.52 0) (layer Eco1.User) (width 0.4))
     (fp_line (start 40.64 12.5) (end 40.64 14) (layer F.CrtYd) (width 0.1))
     (fp_line (start -8.89 9.96) (end -8.89 12.5) (layer F.CrtYd) (width 0.1))
@@
     (fp_line (start -8.89 9.96) (end -8.89 12.5) (layer F.Fab) (width 0.2))
     (fp_circle (center 33.02 0) (end 36.52 0) (layer Dwgs.User) (width 0.2))
-    (fp_circle (center 33.02 0) (end 36.72 0) (layer Eco1.User) (width 0.4))
+    (fp_circle (center 33.02 0) (end 36.62 0) (layer Eco1.User) (width 0.4))
     (fp_circle (center 33.02 0) (end 36.02 0) (layer Dwgs.User) (width 0.2))
     (fp_line (start 40.52 4) (end 40.52 12.5) (layer Dwgs.User) (width 0.2))
@@
     (fp_line (start -7.3 -1.4) (end -7.3 1.4) (layer Dwgs.User) (width 0.2))
     (fp_line (start -7.5 12.5) (end 7.5 12.5) (layer Dwgs.User) (width 0.2))
-    (fp_circle (center 0 0) (end 3.7 0) (layer Eco1.User) (width 0.4))
+    (fp_circle (center 0 0) (end 3.6 0) (layer Eco1.User) (width 0.4))
     (fp_line (start -40.64 12.5) (end 40.64 12.5) (layer F.Fab) (width 0.2))
     (fp_line (start -40.64 14) (end 40.64 14) (layer F.Fab) (width 0.2))
@@
     (fp_line (start 8.89 9.96) (end 8.89 12.5) (layer F.CrtYd) (width 0.1))
     (fp_line (start 24.13 9.96) (end 24.13 12.5) (layer F.CrtYd) (width 0.1))
-    (fp_circle (center -7.9 0) (end -6.5 0) (layer Eco1.User) (width 0.4))
     (fp_text user PLS-06 (at -16.51 11.23) (layer F.Fab)
       (effects (font (size 1 1) (thickness 0.2)))
@@
       (net 13 VA))
   )
-  (module KCL-TH-SL:SW-PBS-24-302SP-2.5-PNL-13.0 (layer F.Cu)
+  (module KCL-TH-SL:SW-PBS-24-302SP-2.5-PNL-12.0 (layer F.Cu)
     (at 105.41 177.8)
     (fp_text reference SB1 (at 8.89 8.255) (layer F.SilkS)
@@
     (fp_line (start -8.5 -6.75) (end -8.5 6.75) (layer F.CrtYd) (width 0.1))
     (fp_line (start 8.5 -6.75) (end 8.5 6.75) (layer F.CrtYd) (width 0.1))
-    (fp_circle (center 0 0) (end 6.5 0) (layer Eco1.User) (width 0.4))
+    (fp_circle (center 0 0) (end 6 0) (layer Eco1.User) (width 0.4))
     (fp_circle (center 0 0) (end 6 0) (layer F.Fab) (width 0.2))
     (fp_arc (start 0 0) (end 0 -5) (angle 81.3) (layer F.SilkS) (width 0.2))

Commit message: ТКП-1.21.A-2 Fishtaur [REV1A] SM: VE1 cipher changed from ТКП-6.1.1.A1-2 to ТКП-6.1.1.A1.A1.A.1-1, VE2 cipher changed from ТКП-6.1.3.B1-1 to ТКП-6.1.3.A1.B1.2-1.A1.B1
Parts:
- VE1: value ТКП-6.1.1.A1-2 -> ТКП-6.1.1.A1.A1.A.1-1; footprint SBEL:ТКП-6.1.1.A1 -> SBEPL:ТКП-6.1.1.A1.A1.A
- VE2: value ТКП-6.1.3.B1-1 -> ТКП-6.1.3.A1.B1.2-1.A1.B1; footprint SBEL:ТКП-6.1.3 -> SBEPL:ТКП-6.1.3.A1

Commit message: ТКП-1.21.A-2 Fishtaur [REV1A] SM: some changes
Parts:
- HL1: footprint KCL-TH-SL:LED-ROUND-05.0-UNI-SH-SPACER-PNL-5.3 -> KCL-TH-SL:LED-ROUND-05.0-UNI-SH-SPACER-PNL-5.2
- VD2, VD3: value 400x -> 4001
- VD4, VD5: value 34A -> Д9Б
- VE2: value ТКП-6.1.3.A1.B1.2-1.A1.B1 -> ТКП-6.1.3.B1.B2.3-1.A2.B1; footprint SBEPL:ТКП-6.1.3.A1 -> SBEPL:ТКП-6.1.3.B1
Other:
- board text added: "1. SB1 установить на проставку ТКП-3.43.A."
- board text removed: "1. SB1 установить на проставку ТКП-3.35.A."
Changed lines of the file:
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@@
   (title_block
     (title ТКП-1.21.A-2)
-    (date 2025-01-04)
+    (date 2025-06-25)
     (rev 1A)
     (company "Fishtaur [REV1A] SM")
@@
     (add_net VREF)
   )
-  (module SBEPL:ТКП-6.1.3.A1 locked (layer F.Cu)
+  (module SBEPL:ТКП-6.1.3.B1 locked (layer F.Cu)
     (at 105.41 148.59)
     (fp_text reference VE2 (at 0 53.34) (layer F.SilkS) hide
       (effects (font (size 1 1) (thickness 0.2)))
     )
-    (fp_text value ТКП-6.1.3.A1.B1.2-1.A1.B1 (at 0 52.07) (layer F.Fab) hide
-      (effects (font (size 1 1) (thickness 0.2)))
-    )
-    (fp_arc (start -43.9 -56.65) (end -43.9 -59.75) (angle -90) (layer Eco1.User) (width 0.4))
-    (fp_arc (start 43.9 -56.65) (end 47 -56.65) (angle -90) (layer Eco1.User) (width 0.4))
-    (fp_arc (start -43.9 56.65) (end -47 56.65) (angle -90) (layer Eco1.User) (width 0.4))
-    (fp_arc (start 43.9 56.65) (end 43.9 59.75) (angle -90) (layer Eco1.User) (width 0.4))
+    (fp_text value ТКП-6.1.3.B1.B2.3-1.A2.B1 (at 0 52.07) (layer F.Fab) hide
+      (effects (font (size 1 1) (thickness 0.2)))
+    )
+    (fp_line (start 3.3 13.97) (end 3.3 15.865338) (layer Eco1.User) (width 0.4))
+    (fp_line (start -3.3 13.97) (end -3.3 15.865338) (layer Eco1.User) (width 0.4))
     (fp_line (start 47 -56.65) (end 47 56.65) (layer Eco1.User) (width 0.4))
     (fp_line (start -47 -56.65) (end -47 56.65) (layer Eco1.User) (width 0.4))
     (fp_line (start -43.9 59.75) (end 43.9 59.75) (layer Eco1.User) (width 0.4))
     (fp_line (start -43.9 -59.75) (end 43.9 -59.75) (layer Eco1.User) (width 0.4))
-    (fp_circle (center -38.6 -51.35) (end -37.1 -51.35) (layer Eco1.User) (width 0.4))
-    (fp_circle (center 38.6 -51.35) (end 40.1 -51.35) (layer Eco1.User) (width 0.4))
-    (fp_circle (center -38.6 51.35) (end -37.1 51.35) (layer Eco1.User) (width 0.4))
-    (fp_circle (center 38.6 51.35) (end 40.1 51.35) (layer Eco1.User) (width 0.4))
+    (fp_circle (center -38.6 -51.35) (end -36.6 -51.35) (layer Eco1.User) (width 0.4))
+    (fp_circle (center 38.6 -51.35) (end 40.6 -51.35) (layer Eco1.User) (width 0.4))
+    (fp_circle (center -38.6 51.35) (end -36.6 51.35) (layer Eco1.User) (width 0.4))
+    (fp_circle (center 38.6 51.35) (end 40.6 51.35) (layer Eco1.User) (width 0.4))
+    (fp_arc (start 6.4 15.865338) (end 3.3 15.865338) (angle -64.4) (layer Eco1.User) (width 0.4))
+    (fp_arc (start -6.4 15.865338) (end -5.051324 18.656583) (angle -64.4) (layer Eco1.User) (width 0.4))
+    (fp_arc (start 0 13.97) (end 3.3 13.97) (angle -180) (layer Eco1.User) (width 0.4))
+    (fp_arc (start 43.9 56.65) (end 43.9 59.75) (angle -90) (layer Eco1.User) (width 0.4))
+    (fp_arc (start -43.9 56.65) (end -47 56.65) (angle -90) (layer Eco1.User) (width 0.4))
+    (fp_arc (start 43.9 -56.65) (end 47 -56.65) (angle -90) (layer Eco1.User) (width 0.4))
+    (fp_arc (start -43.9 -56.65) (end -43.9 -59.75) (angle -90) (layer Eco1.User) (width 0.4))
+    (fp_arc (start 0 29.21) (end 5.0595 18.6605) (angle 308.8) (layer Eco1.User) (width 0.4))
   )
   (module SBEPL:ТКП-6.1.1.A1.A1.A locked (layer F.Cu)
@@
       (effects (font (size 1 1) (thickness 0.2)))
     )
-    (fp_arc (start 43.4 -87.65) (end 45 -87.65) (angle -90) (layer Eco2.User) (width 0.4))
-    (fp_arc (start -43.4 -87.65) (end -43.4 -89.25) (angle -90) (layer Eco2.User) (width 0.4))
-    (fp_arc (start 43.4 -87.65) (end 46.5 -87.65) (angle -90) (layer Eco2.User) (width 0.4))
-    (fp_arc (start -43.4 -87.65) (end -43.4 -90.75) (angle -90) (layer Eco2.User) (width 0.4))
-    (fp_arc (start 33.425 -62.975) (end 33.8 -62.975) (angle -180) (layer Eco2.User) (width 0.4))
-    (fp_arc (start -33.425 -62.975) (end -33.05 -62.975) (angle -180) (layer Eco2.User) (width 0.4))
-    (fp_arc (start 41.7 49.65) (end 44.8 49.65) (angle -90) (layer Eco2.User) (width 0.4))
-    (fp_arc (start -41.7 49.65) (end -41.7 46.55) (angle -90) (layer Eco2.User) (width 0.4))
-    (fp_arc (start 41.7 -49.65) (end 41.7 -46.55) (angle -90) (layer Eco2.User) (width 0.4))
-    (fp_arc (start -41.7 -49.65) (end -44.8 -49.65) (angle -90) (layer Eco2.User) (width 0.4))
-    (fp_arc (start 36.9 49.65) (end 36.9 46.55) (angle -90) (layer Eco2.User) (width 0.4))
-    (fp_arc (start -36.9 49.65) (end -33.8 49.65) (angle -90) (layer Eco2.User) (width 0.4))
-    (fp_arc (start 36.9 -49.65) (end 33.8 -49.65) (angle -90) (layer Eco2.User) (width 0.4))
-    (fp_arc (start -36.9 -49.65) (end -36.9 -46.55) (angle -90) (layer Eco2.User) (width 0.4))
     (fp_circle (center 38.6 51.35) (end 40.725 51.35) (layer Eco2.User) (width 0.4))
     (fp_circle (center -38.6 51.35) (end -36.475 51.35) (layer Eco2.User) (width 0.4))
@@
     (fp_line (start -33.05 57.75) (end -33.05 59.25) (layer Eco2.User) (width 0.4))
     (fp_line (start 33.05 57.75) (end 33.05 59.25) (layer Eco2.User) (width 0.4))
+    (fp_arc (start 43.4 -87.65) (end 45 -87.65) (angle -90) (layer Eco2.User) (width 0.4))
+    (fp_arc (start -43.4 -87.65) (end -43.4 -89.25) (angle -90) (layer Eco2.User) (width 0.4))
+    (fp_arc (start 43.4 -87.65) (end 46.5 -87.65) (angle -90) (layer Eco2.User) (width 0.4))
+    (fp_arc (start -43.4 -87.65) (end -43.4 -90.75) (angle -90) (layer Eco2.User) (width 0.4))
+    (fp_arc (start 33.425 -62.975) (end 33.8 -62.975) (angle -180) (layer Eco2.User) (width 0.4))
+    (fp_arc (start -33.425 -62.975) (end -33.05 -62.975) (angle -180) (layer Eco2.User) (width 0.4))
+    (fp_arc (start 41.7 49.65) (end 44.8 49.65) (angle -90) (layer Eco2.User) (width 0.4))
+    (fp_arc (start -41.7 49.65) (end -41.7 46.55) (angle -90) (layer Eco2.User) (width 0.4))
+    (fp_arc (start 41.7 -49.65) (end 41.7 -46.55) (angle -90) (layer Eco2.User) (width 0.4))
+    (fp_arc (start -41.7 -49.65) (end -44.8 -49.65) (angle -90) (layer Eco2.User) (width 0.4))
+    (fp_arc (start 36.9 49.65) (end 36.9 46.55) (angle -90) (layer Eco2.User) (width 0.4))
+    (fp_arc (start -36.9 49.65) (end -33.8 49.65) (angle -90) (layer Eco2.User) (width 0.4))
+    (fp_arc (start 36.9 -49.65) (end 33.8 -49.65) (angle -90) (layer Eco2.User) (width 0.4))
+    (fp_arc (start -36.9 -49.65) (end -36.9 -46.55) (angle -90) (layer Eco2.User) (width 0.4))
   )
   (module KCL-TH-SL:CON-PAD-S-1.0-2.0 (layer F.Cu)
@@
       (net 10 /J2))
   )
-  (module KCL-TH-SL:LED-ROUND-05.0-UNI-SH-SPACER-PNL-5.3 (layer F.Cu)
+  (module KCL-TH-SL:LED-ROUND-05.0-UNI-SH-SPACER-PNL-5.2 (layer F.Cu)
     (at 105.41 162.56 90)
     (fp_text reference HL1 (at 3.81 0 180) (layer F.SilkS)
@@
     (fp_circle (center 0 0) (end 2.5 0) (layer F.Fab) (width 0.2))
     (fp_line (start -2.5 -1.466994) (end -2.5 1.466994) (layer F.Fab) (width 0.2))
-    (fp_circle (center 0 0) (end 2.65 0) (layer Eco1.User) (width 0.4))
+    (fp_circle (center 0 0) (end 2.6 0) (layer Eco1.User) (width 0.4))
     (fp_arc (start 0 0) (end -2.5 1.469694) (angle -299.1) (layer F.Fab) (width 0.2))
     (pad C thru_hole circle (at -1.27 0 90) (size 2 2) (drill 0.7) (layers B.Cu B.Mask)
@@
       (effects (font (size 1 1) (thickness 0.2)))
     )
-    (fp_text value DC-005 (at 0 -10.795) (layer F.Fab)
+    (fp_text value DC-005 (at 0 -6.985) (layer F.Fab)
       (effects (font (size 1 1) (thickness 0.2)))
     )
@@
       (effects (font (size 1 1) (thickness 0.2)) (justify left))
     )
-    (fp_text value 34A (at 0 -2.54) (layer F.Fab)
+    (fp_text value Д9Б (at 0 -2.54) (layer F.Fab)
       (effects (font (size 1 1) (thickness 0.2)))
     )
@@
       (effects (font (size 1 1) (thickness 0.2)) (justify left))
     )
-    (fp_text value 34A (at 0 -2.54) (layer F.Fab)
+    (fp_text value Д9Б (at 0 -2.54) (layer F.Fab)
       (effects (font (size 1 1) (thickness 0.2)))
     )
@@
       (effects (font (size 1 1) (thickness 0.2)) (justify right))
     )
-    (fp_text value 400x (at 0 0) (layer F.Fab)
+    (fp_text value 4001 (at 0 0) (layer F.Fab)
       (effects (font (size 1 1) (thickness 0.2)))
     )
@@
       (effects (font (size 1 1) (thickness 0.2)) (justify right))
     )
-    (fp_text value 400x (at 0 0) (layer F.Fab)
+    (fp_text value 4001 (at 0 0) (layer F.Fab)
       (effects (font (size 1 1) (thickness 0.2)))
     )
@@
     (effects (font (size 2.54 2.54) (thickness 0.2)) (justify left))
   )
-  (gr_text "1. SB1 установить на проставку ТКП-3.35.A." (at 90.17 246.38) (layer F.Fab)
+  (gr_text "1. SB1 установить на проставку ТКП-3.43.A." (at 90.17 246.38) (layer F.Fab)
     (effects (font (size 2.54 2.54) (thickness 0.2)) (justify left))
   )
