File: PCBS-PCAS/ТКП-3.21.A/ТКП-1.21.A-1/ТКП-1.21.A-1.kicad_pcb (KiCad board)
At the start: 2 copper layers, 86.4 x 95.3 mm, 81 parts, among them J1 0.6, J2 0.6, J3 0.6, J4 0.6, X1 +, X2 -, X3 COM

Commit message: ТКП-1.21.A-1 Fishtaur [REV1A]: some changes
Parts:
- VD2, VD3: value 400x -> 4001
- VD4, VD5: value 34A -> Д9Б
