File: PCBS-PCAS/ТКП-3.40.A/ТКП-1.38.A-2/ТКП-1.38.A-2.kicad_pcb (KiCad board)
At the start: 2 copper layers, 58.4 x 81.3 mm, 121 parts, among them J1 X, J10 X, J11 0, J12 X, J13 0, J14 0, J2 0, J3 0, J4 0, J5 0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

Commit message: ТКП-1.38.A-2 Great Depression Phaser [REV1A] SM: minor changes
Parts:
- added VE2: ТКП-6.2.4.A1.B1.4-1.A2.B1, SBEPL:ТКП-6.2.4.A1, F.Cu at (105.4, 148.6)
- VE1: value 1590N1 -> ТКП-6.2.1.A1.A1.A.1-1; footprint SBEL:1590N1_A1 -> SBEPL:ТКП-6.2.1.A1.A1.A

Commit message: ТКП-1.38.A-2 Great Depression Phaser [REV1A] SM: minor changes
Parts:
- HL1: footprint KCL-TH-ML:LED-ROUND-05.0-UNI-SH-SPACER-PNL-5.3 -> KCL-TH-ML:LED-ROUND-05.0-UNI-SH-SPACER-PNL-6.6
- RPB1: footprint SBKCL-TH-ML:RPB-1590N1-18-2x17-OR-2x1x17-1.6-PNL-7.4-2.8 -> SBKCL-TH-ML:RPB-1590N1-18-2x17-OR-2x1x17-1.6-PNL-7.2
- SB1: footprint KCL-TH-ML:SW-PBS-24-302SP-2.5-PNL-13.0 -> KCL-TH-ML:SW-PBS-24-302SP-2.5-PNL-12.0
